File: Circuit/v4.sch (KiCad schematic (older format))
At the start: 38 parts, among them J1 Battery, J2 AVR-ISP-6, J3 TX Connector, J4 RX Connector, J5 Alt Battery, J6 Alt RX Conn, J7 Alt TX Conn, J8 Remote temp input 47K @ 25oC, Q1 IRLML6244TRPBF, U1 EL3H7(B)(TA)-VG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

Commit message: Change Opto to HMHA2801
Parts:
- U1: value EL3H7(B)(TA)-VG -> HMHA2801
Changed lines of the file:
@@
 P 9190 4790
 F 0 "U1" H 9190 5115 50  0000 C CNN
-F 1 "EL3H7(B)(TA)-VG" H 9190 5024 50  0000 C CNN
+F 1 "HMHA2801" H 9190 5024 50  0000 C CNN
 F 2 "Housings_SSOP:SOP-4_4.4x2.8mm_Pitch1.27mm" H 8990 4590 50  0001 L CIN
-F 3 "https://www.digikey.co.uk/product-detail/en/everlight-electronics-co-ltd/EL3H7-B-TA-VG/1080-1197-1-ND/2675931" H 9190 4790 50  0001 L CNN
+F 3 "https://www.mouser.co.uk/datasheet/2/308/HMHA2801-1306522.pdf" H 9190 4790 50  0001 L CNN
 	1    9190 4790
 	1    0    0    -1

Commit message: Optocoupler changes
Parts:
- U1: symbol EL3H7-G:EL3H7-G -> Isolator:PC817
Changed lines of the file:
@@
 PA7 has a higher current output than other pins
 $Comp
-L EL3H7-G:EL3H7-G U1
+L Isolator:PC817 U1
 U 1 1 5BF1DCDE
 P 9190 4790

Commit message: upgrde to kicad 5.1
Parts:
- U4: symbol MCU_Microchip_ATtiny:ATtiny841-SSU -> v4-rescue:ATtiny841-SSU-MCU_Microchip_ATtiny
Changed lines of the file:
@@
 EESchema Schematic File Version 4
 LIBS:v4-cache
-EELAYER 26 0
+EELAYER 29 0
 EELAYER END
 $Descr A4 11693 8268
@@
 $EndDescr
 $Comp
-L MCU_Microchip_ATtiny:ATtiny841-SSU U4
+L v4-rescue:ATtiny841-SSU-MCU_Microchip_ATtiny U4
 U 1 1 5BC63D51
 P 1650 3670

Commit message: Updated circuit with 510 ohm gate current limit resistor
Parts:
- added R14: 510R, Resistors_SMD:R_0805_HandSoldering, symbol Device:R
- J8: footprint Pin_Headers:Pin_Header_Straight_1x04_Pitch2.54mm -> Pin_Headers:Pin_Header_Straight_1x05_Pitch2.54mm; symbol Connector:Conn_01x04_Male -> Connector:Conn_01x05_Male
- R15: value 47K YAGEO RC0805FR-0747KL -> 10K
Connections:
- wire segments 138 -> 139
Changed lines of the file:
@@
 P 7780 3560
 F 0 "R15" H 7850 3606 50  0000 L CNN
-F 1 "47K YAGEO RC0805FR-0747KL" H 6550 3430 50  0000 L CNN
+F 1 "10K" H 7560 3560 50  0000 L CNN
 F 2 "Resistors_SMD:R_0805_HandSoldering" V 7710 3560 50  0001 C CNN
 F 3 "YAGEO RC0805FR-0747KL" H 7780 3560 50  0001 C CNN
@@
 Wire Wire Line
 	2790 3370 2250 3370
-Text GLabel 7360 3580 0    50   Input ~ 0
+Text GLabel 7060 3580 0    50   Input ~ 0
 DUMP_LOAD_ENABLE
 Wire Wire Line
@@
 	4280 6330 4280 6190
 $Comp
-L Connector:Conn_01x04_Male J8
+L Connector:Conn_01x05_Male J8
 U 1 1 5BF61617
-P 4870 5750
-F 0 "J8" H 4843 5630 50  0000 R CNN
-F 1 "Remote temp input 47K @ 25oC" H 4850 5990 50  0000 R CNN
-F 2 "Pin_Headers:Pin_Header_Straight_1x04_Pitch2.54mm" H 4870 5750 50  0001 C CNN
-F 3 "~" H 4870 5750 50  0001 C CNN
-	1    4870 5750
+P 4870 5650
+F 0 "J8" H 4843 5530 50  0000 R CNN
+F 1 "Remote temp input 47K @ 25oC" H 4850 5890 50  0000 R CNN
+F 2 "Pin_Headers:Pin_Header_Straight_1x05_Pitch2.54mm" H 4870 5650 50  0001 C CNN
+F 3 "~" H 4870 5650 50  0001 C CNN
+	1    4870 5650
 	-1   0    0    1
 $EndComp
@@
 Wire Wire Line
 	950  4570 950  4590
+$Comp
+L Device:R R14
+U 1 1 5CB1F559
+P 7210 3580
+F 0 "R14" H 7280 3626 50  0000 L CNN
+F 1 "510R" H 7280 3520 50  0000 L CNN
+F 2 "Resistors_SMD:R_0805_HandSoldering" V 7140 3580 50  0001 C CNN
+F 3 "" H 7210 3580 50  0001 C CNN
+	1    7210 3580
+	0    1    1    0
+$EndComp
+$Comp
+L power:GND #PWR?
+U 1 1 5CB35AE2
+P 4090 5450
+F 0 "#PWR?" H 4090 5200 50  0001 C CNN
+F 1 "GND" H 4095 5277 50  0000 C CNN
+F 2 "" H 4090 5450 50  0001 C CNN
+F 3 "" H 4090 5450 50  0001 C CNN
+	1    4090 5450
+	1    0    0    -1
+$EndComp
+Wire Wire Line
+	4670 5450 4090 5450
 $EndSCHEMATC

Commit message: Added 10uF cap to charge MOSFET slower to prevent fast switch on currents resetting MCU
Parts:
- added C3: 10uF 10V, Capacitors_SMD:C_0805_HandSoldering, symbol Device:C
- R15: value 10K -> 47K
Connections:
- wire segments 139 -> 141
Changed lines of the file:
@@
 P 7780 3560
 F 0 "R15" H 7850 3606 50  0000 L CNN
-F 1 "10K" H 7560 3560 50  0000 L CNN
+F 1 "47K" H 7850 3520 50  0000 L CNN
 F 2 "Resistors_SMD:R_0805_HandSoldering" V 7710 3560 50  0001 C CNN
 F 3 "YAGEO RC0805FR-0747KL" H 7780 3560 50  0001 C CNN
@@
 Wire Wire Line
 	2790 3370 2250 3370
-Text GLabel 7060 3580 0    50   Input ~ 0
+Text GLabel 6780 3580 0    50   Input ~ 0
 DUMP_LOAD_ENABLE
 Wire Wire Line
-	7780 3410 7360 3410
-Wire Wire Line
-	7360 3410 7360 3580
+	7780 3410 7500 3410
+Wire Wire Line
+	7360 3410 7080 3580
 Connection ~ 7780 3410
 $Comp
@@
 L Device:R R14
 U 1 1 5CB1F559
-P 7210 3580
-F 0 "R14" H 7280 3626 50  0000 L CNN
-F 1 "510R" H 7280 3520 50  0000 L CNN
-F 2 "Resistors_SMD:R_0805_HandSoldering" V 7140 3580 50  0001 C CNN
-F 3 "" H 7210 3580 50  0001 C CNN
-	1    7210 3580
+P 6930 3580
+F 0 "R14" H 7000 3626 50  0000 L CNN
+F 1 "510R" H 7000 3520 50  0000 L CNN
+F 2 "Resistors_SMD:R_0805_HandSoldering" V 6860 3580 50  0001 C CNN
+F 3 "" H 6930 3580 50  0001 C CNN
+	1    6930 3580
 	0    1    1    0
 $EndComp
 $Comp
-L power:GND #PWR?
+L power:GND #PWR0117
 U 1 1 5CB35AE2
 P 4090 5450
-F 0 "#PWR?" H 4090 5200 50  0001 C CNN
+F 0 "#PWR0117" H 4090 5200 50  0001 C CNN
 F 1 "GND" H 4095 5277 50  0000 C CNN
 F 2 "" H 4090 5450 50  0001 C CNN
@@
 Wire Wire Line
 	4670 5450 4090 5450
+$Comp
+L Device:C C3
+U 1 1 5CB3BB54
+P 7500 3560
+F 0 "C3" H 7360 3560 50  0000 R CNN
+F 1 "10uF 10V" H 7390 3460 50  0000 R CNN
+F 2 "Capacitors_SMD:C_0805_HandSoldering" H 7538 3410 50  0001 C CNN
+F 3 "https://datasheet.lcsc.com/szlcsc/YAGEO-CC0805KRX5R6BB106_C272880.pdf" H 7500 3560 50  0001 C CNN
+	1    7500 3560
+	1    0    0    -1
+$EndComp
+Connection ~ 7500 3410
+Wire Wire Line
+	7500 3410 7360 3410
+Wire Wire Line
+	7500 3710 7780 3710
 $EndSCHEMATC

Commit message: Updates to circuit design and layout
Parts:
- removed J5: Alt Battery, Pin_Headers:Pin_Header_Straight_1x02_Pitch2.54mm, symbol Connector:Conn_01x02_Male
- removed J6: Alt RX Conn, Pin_Headers:Pin_Header_Straight_1x02_Pitch2.54mm, symbol Connector:Conn_01x02_Male
- removed J7: Alt TX Conn, Pin_Headers:Pin_Header_Straight_1x02_Pitch2.54mm, symbol Connector:Conn_01x02_Male
- removed TP1: TestPoint, TestPoint:TestPoint_Pad_2.0x2.0mm, symbol Connector:TestPoint
- R10, R12, R8: value 2R2 1W -> 2R2 1W
Connections:
- wire segments 141 -> 121
Changed lines of the file:
@@
 	950  2610 950  2730
-Wire Wire Line
-	950  3030 950  4570
 Wire Wire Line
 	950  4590 1650 4590
@@
 Wire Wire Line
 	2120 6230 2250 6230
-Wire Wire Line
-	1670 1450 1750 1450
 $Comp
 L power:GND #PWR0105
@@
 	1    0    0    -1
 $EndComp
-Wire Wire Line
-	1670 1350 1720 1350
 Wire Wire Line
 	1770 1100 1770 1350
@@
 $EndComp
 Wire Wire Line
-	9490 4690 9630 4690
-Wire Wire Line
 	9740 4690 9740 4730
-Wire Wire Line
-	9490 4890 9590 4890
 Wire Wire Line
 	9740 4890 9740 4830
@@
 P 7100 2700
 F 0 "R8" H 7170 2746 50  0000 L CNN
-F 1 "2R2  1W" H 7170 2655 50  0000 L CNN
+F 1 "2R2 1W" H 7170 2655 50  0000 L CNN
 F 2 "Resistors_SMD:R_2512" V 7030 2700 50  0001 C CNN
 F 3 "https://datasheet.lcsc.com/szlcsc/Ever-Ohms-Tech-CR2512F2R2E04_C147074.pdf" H 7100 2700 50  0001 C CNN
@@
 P 7450 2700
 F 0 "R10" H 7520 2746 50  0000 L CNN
-F 1 "2R2  1W" H 7520 2655 50  0000 L CNN
+F 1 "2R2 1W" H 7520 2655 50  0000 L CNN
 F 2 "Resistors_SMD:R_2512" V 7380 2700 50  0001 C CNN
 F 3 "https://datasheet.lcsc.com/szlcsc/Ever-Ohms-Tech-CR2512F2R2E04_C147074.pdf" H 7450 2700 50  0001 C CNN
@@
 P 7800 2700
 F 0 "R12" H 7870 2746 50  0000 L CNN
-F 1 "2R2  1W" H 7870 2655 50  0000 L CNN
+F 1 "2R2 1W" H 7870 2655 50  0000 L CNN
 F 2 "Resistors_SMD:R_2512" V 7730 2700 50  0001 C CNN
 F 3 "https://datasheet.lcsc.com/szlcsc/Ever-Ohms-Tech-CR2512F2R2E04_C147074.pdf" H 7800 2700 50  0001 C CNN
@@
 $EndComp
 Wire Wire Line
-	8690 5460 8600 5460
-Wire Wire Line
 	8320 5460 8320 5380
 $Comp
@@
 	7980 5560 8250 5560
 Connection ~ 8250 5560
-Wire Wire Line
-	8250 5560 8520 5560
 $Comp
 L Device:LED D3
@@
 	3050 3750 3050 3670
 $Comp
-L Connector:Conn_01x02_Male J6
-U 1 1 5BF7620E
-P 8890 5860
-F 0 "J6" H 8863 5740 50  0000 R CNN
-F 1 "Alt RX Conn" H 8863 5831 50  0000 R CNN
-F 2 "Pin_Headers:Pin_Header_Straight_1x02_Pitch2.54mm" H 8890 5860 50  0001 C CNN
-F 3 "~" H 8890 5860 50  0001 C CNN
-	1    8890 5860
-	-1   0    0    1
-$EndComp
-Wire Wire Line
-	8690 5760 8600 5760
-Wire Wire Line
-	8600 5760 8600 5460
-Connection ~ 8600 5460
-Wire Wire Line
-	8600 5460 8320 5460
-Wire Wire Line
-	8520 5560 8520 5860
-Wire Wire Line
-	8520 5860 8690 5860
-Connection ~ 8520 5560
-Wire Wire Line
-	8520 5560 8690 5560
-$Comp
-L Connector:Conn_01x02_Male J7
-U 1 1 5BF806EA
-P 9940 5070
-F 0 "J7" H 9912 4950 50  0000 R CNN
-F 1 "Alt TX Conn" H 9912 5041 50  0000 R CNN
-F 2 "Pin_Headers:Pin_Header_Straight_1x02_Pitch2.54mm" H 9940 5070 50  0001 C CNN
-F 3 "~" H 9940 5070 50  0001 C CNN
-	1    9940 5070
-	-1   0    0    1
-$EndComp
-Wire Wire Line
-	9740 4970 9630 4970
-Wire Wire Line
-	9630 4970 9630 4690
-Connection ~ 9630 4690
-Wire Wire Line
-	9630 4690 9740 4690
-Wire Wire Line
-	9590 4890 9590 5070
-Wire Wire Line
-	9590 5070 9740 5070
-Connection ~ 9590 4890
-Wire Wire Line
-	9590 4890 9740 4890
-$Comp
-L Connector:Conn_01x02_Male J5
-U 1 1 5BF86BF7
-P 1480 1740
-F 0 "J5" H 1586 1918 50  0000 C CNN
-F 1 "Alt Battery" H 1586 1827 50  0000 C CNN
-F 2 "Pin_Headers:Pin_Header_Straight_1x02_Pitch2.54mm" H 1480 1740 50  0001 C CNN
-F 3 "~" H 1480 1740 50  0001 C CNN
-	1    1480 1740
-	1    0    0    -1
-$EndComp
-Wire Wire Line
-	1680 1740 1720 1740
-Wire Wire Line
-	1720 1740 1720 1350
-Connection ~ 1720 1350
-Wire Wire Line
-	1720 1350 1770 1350
-Wire Wire Line
-	1750 1450 1750 1840
-Wire Wire Line
-	1750 1840 1680 1840
-Connection ~ 1750 1450
-$Comp
 L Connector:TestPoint TP2
 U 1 1 5BF9C005
@@
 Wire Wire Line
 	2250 3070 3020 3070
-Wire Wire Line
-	1750 1450 2040 1450
 Connection ~ 2040 1450
 Connection ~ 1870 1100
@@
 Wire Wire Line
 	4670 5550 4560 5550
-$Comp
-L Connector:TestPoint TP1
-U 1 1 5C2982C3
-P 780 4570
-F 0 "TP1" H 700 4760 50  0000 L CNN
-F 1 "TestPoint" H 570 4520 50  0000 L CNN
-F 2 "TestPoint:TestPoint_Pad_2.0x2.0mm" H 980 4570 50  0001 C CNN
-F 3 "~" H 980 4570 50  0001 C CNN
-	1    780  4570
-	1    0    0    -1
-$EndComp
-Wire Wire Line
-	780  4570 950  4570
-Connection ~ 950  4570
-Wire Wire Line
-	950  4570 950  4590
 $Comp
 L Device:R R14
@@
 L power:GND #PWR0117
 U 1 1 5CB35AE2
-P 4090 5450
-F 0 "#PWR0117" H 4090 5200 50  0001 C CNN
-F 1 "GND" H 4095 5277 50  0000 C CNN
-F 2 "" H 4090 5450 50  0001 C CNN
-F 3 "" H 4090 5450 50  0001 C CNN
-	1    4090 5450
-	1    0    0    -1
-$EndComp
-Wire Wire Line
-	4670 5450 4090 5450
+P 4410 5280
+F 0 "#PWR0117" H 4410 5030 50  0001 C CNN
+F 1 "GND" H 4415 5107 50  0000 C CNN
+F 2 "" H 4410 5280 50  0001 C CNN
+F 3 "" H 4410 5280 50  0001 C CNN
+	1    4410 5280
+	1    0    0    -1
+$EndComp
+Wire Wire Line
+	4670 5450 4410 5280
 $Comp
 L Device:C C3
@@
 Wire Wire Line
 	7500 3710 7780 3710
+Wire Wire Line
+	950  3030 950  4590
+Wire Wire Line
+	9490 4690 9740 4690
+Wire Wire Line
+	9490 4890 9740 4890
+Wire Wire Line
+	8320 5460 8690 5460
+Wire Wire Line
+	8250 5560 8690 5560
+Wire Wire Line
+	1670 1350 1770 1350
+Wire Wire Line
+	1670 1450 2040 1450
 $EndSCHEMATC

Commit message: Major tidy up and initial BOM
Parts:
- U4: symbol v4-rescue:ATtiny841-SSU-MCU_Microchip_ATtiny -> v4-rescue:ATtiny841-SSU-MCU_Microchip_ATtiny-v4-rescue
Changed lines of the file:
@@
 $EndDescr
 $Comp
-L v4-rescue:ATtiny841-SSU-MCU_Microchip_ATtiny U4
+L v4-rescue:ATtiny841-SSU-MCU_Microchip_ATtiny-v4-rescue U4
 U 1 1 5BC63D51
 P 1650 3670
@@
 F 1 "HMHA2801" H 9190 5024 50  0000 C CNN
 F 2 "Housings_SSOP:SOP-4_4.4x2.8mm_Pitch1.27mm" H 8990 4590 50  0001 L CIN
-F 3 "https://www.mouser.co.uk/datasheet/2/308/HMHA2801-1306522.pdf" H 9190 4790 50  0001 L CNN
+F 3 "https://uk.farnell.com/on-semiconductor/hmha2801/optocoupler-single-channel/dp/1652504" H 9190 4790 50  0001 L CNN
 	1    9190 4790
 	1    0    0    -1

Commit message: Updated datasheet link
Parts:
- R19: value Thermistor Sunlord SDNT2012X473F4150FTF -> SDNT2012X473F4150FTF
Changed lines of the file:
@@
 F 1 "Battery" H 1576 1437 50  0000 C CNN
 F 2 "Connectors_JST:JST_PH_S2B-PH-K_02x2.00mm_Angled" H 1470 1350 50  0001 C CNN
-F 3 "~" H 1470 1350 50  0001 C CNN
+F 3 "http://www.farnell.com/datasheets/2057211.pdf" H 1470 1350 50  0001 C CNN
 	1    1470 1350
 	1    0    0    -1
@@
 F 1 "RX Connector" H 8863 5531 50  0000 R CNN
 F 2 "Connectors_JST:JST_PH_S2B-PH-K_02x2.00mm_Angled" H 8890 5560 50  0001 C CNN
-F 3 "~" H 8890 5560 50  0001 C CNN
+F 3 "http://www.farnell.com/datasheets/2057211.pdf" H 8890 5560 50  0001 C CNN
 	1    8890 5560
 	-1   0    0    1
@@
 P 2740 6590
 F 0 "R19" H 2810 6636 50  0000 L CNN
-F 1 "Thermistor Sunlord SDNT2012X473F4150FTF" H 2810 6530 50  0000 L CNN
+F 1 "SDNT2012X473F4150FTF" H 2810 6530 50  0000 L CNN
 F 2 "Resistors_SMD:R_0805_HandSoldering" V 2670 6590 50  0001 C CNN
 F 3 "https://datasheet.lcsc.com/szlcsc/Sunlord-SDNT2012X473F4150FTF_C95969.pdf" H 2740 6590 50  0001 C CNN
