File: Circuit/v4.sch (KiCad schematic (older format))
At the start: 37 parts, among them J2 AVR-ISP-6, Q1 IRLML6244TRPBF, U1 HMHA2801, U4 ATtiny841-SSU

Commit message: Change of dimensions and layout board is now 30x49mm
Parts:
- R22: footprint Resistors_THT:R_Axial_Power_L25.0mm_W9.0mm_P30.48mm -> Resistors_THT:R_Axial_Power_L25.0mm_W9.0mm_P27.94mm
Changed lines of the file:
@@
 F 0 "R22" V 7463 1050 50  0000 C CNN
 F 1 "4R4" V 7554 1050 50  0000 C CNN
-F 2 "Resistors_THT:R_Axial_Power_L25.0mm_W9.0mm_P30.48mm" V 7600 1050 50  0001 C CNN
+F 2 "Resistors_THT:R_Axial_Power_L25.0mm_W9.0mm_P27.94mm" V 7600 1050 50  0001 C CNN
 F 3 "~" H 7670 1050 50  0001 C CNN
 	1    7670 1050

Commit message: Moved red led onto dump load circuit to free up IO pin
Changed lines of the file:
@@
 Wire Wire Line
 	8050 1990 8100 1990
-Text Notes 6700 1560 0    50   ~ 0
+Text Notes 5990 1620 0    50   ~ 0
 Each row is 8R8 and 4W max (needs to carry 2W @ 4.2V), drops about 470mA.\n
 $Comp
@@
 Wire Wire Line
 	8050 2290 8100 2290
-Text Notes 6710 1430 0    50   ~ 0
+Text Notes 5980 1780 0    50   ~ 0
 Ever Ohms Tech CR2512F2R2E04\nhttps://lcsc.com/product-detail/Chip-Resistor-Surface-Mount_Ever-Ohms-Tech-CR2512F2R2E04_C147074.html\n
 $Comp
@@
 L Device:LED D3
 U 1 1 5BF65B89
-P 4310 3130
-F 0 "D3" H 4450 3230 50  0000 C CNN
-F 1 "RED LED" H 4400 3030 50  0000 C CNN
-F 2 "LEDs:LED_0805_HandSoldering" H 4310 3130 50  0001 C CNN
-F 3 "~" H 4310 3130 50  0001 C CNN
-	1    4310 3130
+P 7980 1350
+F 0 "D3" H 8120 1450 50  0000 C CNN
+F 1 "RED LED" H 8070 1250 50  0000 C CNN
+F 2 "LEDs:LED_0805_HandSoldering" H 7980 1350 50  0001 C CNN
+F 3 "~" H 7980 1350 50  0001 C CNN
+	1    7980 1350
 	-1   0    0    1
 $EndComp
@@
 L Device:R R17
 U 1 1 5BF65CB1
-P 4690 3130
-F 0 "R17" V 4780 3180 50  0000 L CNN
-F 1 "2K2" V 4780 3010 50  0000 L CNN
-F 2 "Resistors_SMD:R_0805_HandSoldering" V 4620 3130 50  0001 C CNN
-F 3 "~" H 4690 3130 50  0001 C CNN
-	1    4690 3130
+P 8360 1350
+F 0 "R17" V 8450 1400 50  0000 L CNN
+F 1 "2K2" V 8450 1230 50  0000 L CNN
+F 2 "Resistors_SMD:R_0805_HandSoldering" V 8290 1350 50  0001 C CNN
+F 3 "~" H 8360 1350 50  0001 C CNN
+	1    8360 1350
 	0    1    1    0
 $EndComp
 Wire Wire Line
-	4460 3130 4540 3130
+	8130 1350 8210 1350
 $Comp
 L Device:LED D4
@@
 $EndComp
 Wire Wire Line
-	4840 3130 4840 3370
-Wire Wire Line
 	4840 3370 5130 3370
 Wire Wire Line
 	5130 3370 5130 3510
-Connection ~ 4840 3370
-Wire Wire Line
-	3870 3570 3870 3130
-Wire Wire Line
-	3870 3130 4160 3130
-Connection ~ 3180 3570
+Wire Wire Line
+	7540 1350 7830 1350
 Wire Wire Line
 	3790 3750 3790 3630
@@
 	7310 6070 7600 6070
 Wire Wire Line
-	3180 3570 3870 3570
-Wire Wire Line
 	3050 3750 3790 3750
 Wire Wire Line
@@
 $EndComp
 Wire Wire Line
-	8510 2160 8510 1050
+	8510 2160 8510 1350
 Wire Wire Line
 	8510 1050 7820 1050
@@
 	1    0    0    -1
 $EndComp
-Wire Wire Line
-	7370 1050 7520 1050
 Text Notes 6640 760  0    50   ~ 0
 Either the SMD or larger power resistor is used - NOT BOTH!\n
+Connection ~ 8510 1350
+Wire Wire Line
+	8510 1350 8510 1050
+Wire Wire Line
+	7540 1350 7540 1050
+Wire Wire Line
+	7370 1050 7520 1050
+Connection ~ 7520 1050
+Wire Wire Line
+	7520 1050 7540 1050
 $EndSCHEMATC

Commit message: Added blue led as optional extra
Parts:
- added D2: Blue, LEDs:LED_0805, symbol Device:LED
- added R23: 2K2, Resistors_SMD:R_0805, symbol Device:R
- D4: value Green LED -> Green
Connections:
- wire segments 125 -> 132
Changed lines of the file:
@@
 P 4310 3370
 F 0 "D4" H 4450 3470 50  0000 C CNN
-F 1 "Green LED" H 4340 3540 50  0000 C CNN
+F 1 "Green" H 4340 3540 50  0000 C CNN
 F 2 "LEDs:LED_0805_HandSoldering" H 4310 3370 50  0001 C CNN
 F 3 "~" H 4310 3370 50  0001 C CNN
@@
 Wire Wire Line
 	7520 1050 7540 1050
+$Comp
+L Device:LED D2
+U 1 1 5CCBC109
+P 4750 2930
+F 0 "D2" H 4890 3030 50  0000 C CNN
+F 1 "Blue" H 4780 3100 50  0000 C CNN
+F 2 "LEDs:LED_0805" H 4750 2930 50  0001 C CNN
+F 3 "~" H 4750 2930 50  0001 C CNN
+	1    4750 2930
+	-1   0    0    1
+$EndComp
+$Comp
+L Device:R R23
+U 1 1 5CCBC10F
+P 5130 2930
+F 0 "R23" V 5220 2980 50  0000 L CNN
+F 1 "2K2" V 5220 2810 50  0000 L CNN
+F 2 "Resistors_SMD:R_0805" V 5060 2930 50  0001 C CNN
+F 3 "~" H 5130 2930 50  0001 C CNN
+	1    5130 2930
+	0    1    1    0
+$EndComp
+Wire Wire Line
+	4900 2930 4980 2930
+$Comp
+L power:GND #PWR02
+U 1 1 5CCBC116
+P 5570 3070
+F 0 "#PWR02" H 5570 2820 50  0001 C CNN
+F 1 "GND" H 5575 2897 50  0000 C CNN
+F 2 "" H 5570 3070 50  0001 C CNN
+F 3 "" H 5570 3070 50  0001 C CNN
+	1    5570 3070
+	1    0    0    -1
+$EndComp
+Wire Wire Line
+	5280 2930 5570 2930
+Wire Wire Line
+	5570 2930 5570 3070
+Wire Wire Line
+	4450 3190 4450 2930
+Wire Wire Line
+	4450 2930 4600 2930
+Wire Wire Line
+	4450 3190 3180 3190
+Wire Wire Line
+	3180 3190 3180 3570
+Connection ~ 3180 3570
 $EndSCHEMATC

Commit message: Indicator blue LED is optional, remove TP2
Parts:
- removed TP2: TestPoint, TestPoint:TestPoint_Pad_2.0x2.0mm, symbol Connector:TestPoint
Connections:
- wire segments 132 -> 131
Other:
- note added: "Blue LED and Resistor are OPTIONAL!"
Changed lines of the file:
@@
 	3050 3750 3050 3670
-$Comp
-L Connector:TestPoint TP2
-U 1 1 5BF9C005
-P 3940 4170
-F 0 "TP2" H 3860 4360 50  0000 L CNN
-F 1 "TestPoint" H 3730 4120 50  0000 L CNN
-F 2 "TestPoint:TestPoint_Pad_2.0x2.0mm" H 4140 4170 50  0001 C CNN
-F 3 "~" H 4140 4170 50  0001 C CNN
-	1    3940 4170
-	1    0    0    -1
-$EndComp
-Wire Wire Line
-	3940 4170 4280 4170
 $Comp
 L Device:Thermistor R19
@@
 Text GLabel 4560 5550 0    50   Input ~ 0
 ENABLE
-Connection ~ 3940 4170
-Wire Wire Line
-	2250 4170 3940 4170
 Text Notes 8150 3920 0    50   ~ 0
 Optocoupler, Phototransistor Output,\n4-SSOP
@@
 	3180 3190 3180 3570
 Connection ~ 3180 3570
+Wire Wire Line
+	2250 4170 4280 4170
+Text Notes 4560 2810 0    50   ~ 0
+Blue LED and Resistor are OPTIONAL!
 $EndSCHEMATC

Commit message: Bill Of Material for LCSC
Parts:
- C2: symbol Device:CP -> Device:C
- R22: value 4R4 -> 10R
Other:
- note added: "Either the SMD or larger power resistor is used - NOT BOTH !\nNote you must pick a resistor with correct power rating!"
- note removed: "Either the SMD or larger power resistor is used - NOT BOTH!\n"
Changed lines of the file:
@@
 F 1 "100nF" H 836 2835 50  0000 R CNN
 F 2 "Capacitors_SMD:C_0805_HandSoldering" H 988 2730 50  0001 C CNN
-F 3 "~" H 950 2880 50  0001 C CNN
+F 3 "https://lcsc.com/product-detail/Multilayer-Ceramic-Capacitors-MLCC-SMD-SMT_100nF-104-10-50V_C49678.html" H 950 2880 50  0001 C CNN
 	1    950  2880
 	1    0    0    -1
@@
 F 1 "Battery" H 6846 6057 50  0000 C CNN
 F 2 "Connectors_JST:JST_PH_S2B-PH-K_02x2.00mm_Angled" H 6740 5970 50  0001 C CNN
-F 3 "http://www.farnell.com/datasheets/2057211.pdf" H 6740 5970 50  0001 C CNN
+F 3 "https://datasheet.lcsc.com/szlcsc/JST-Sales-America-S2B-PH-K-S-LF-SN_C173752.pdf" H 6740 5970 50  0001 C CNN
 	1    6740 5970
 	1    0    0    -1
@@
 F 1 "10K" V 2444 4410 50  0000 C CNN
 F 2 "Resistors_SMD:R_0805_HandSoldering" V 2490 4410 50  0001 C CNN
-F 3 "~" H 2560 4410 50  0001 C CNN
+F 3 "RC0805FR-0710KL" H 2560 4410 50  0001 C CNN
 	1    2560 4410
 	0    1    1    0
@@
 F 1 "AVR-ISP-6" H 1440 6135 50  0000 R CNN
 F 2 "Pin_Headers:Pin_Header_Straight_2x03_Pitch2.54mm" V 1470 6180 50  0001 C CNN
-F 3 " ~" H 445 5580 50  0001 C CNN
+F 3 "https://lcsc.com/product-detail/Pin-Header-Female-Header_Boom-Precision-Elec-2-54mm-2-3P-Header_C65114.html" H 445 5580 50  0001 C CNN
 	1    1720 6130
 	1    0    0    -1
@@
 F 1 "1K" H 3430 2265 50  0000 L CNN
 F 2 "Resistors_SMD:R_0805_HandSoldering" V 3290 2310 50  0001 C CNN
-F 3 "~" H 3360 2310 50  0001 C CNN
+F 3 "RC0805FR-071KL" H 3360 2310 50  0001 C CNN
 	1    3360 2310
 	1    0    0    -1
@@
 	3360 2580 3360 2460
 $Comp
-L Device:CP C2
+L Device:C C2
 U 1 1 5D1FC233
 P 4140 2730
@@
 F 1 "2.2uF" H 4258 2685 50  0000 L CNN
 F 2 "Capacitors_SMD:C_0805_HandSoldering" H 4178 2580 50  0001 C CNN
-F 3 "~" H 4140 2730 50  0001 C CNN
+F 3 "https://lcsc.com/product-detail/Multilayer-Ceramic-Capacitors-MLCC-SMD-SMT_2-2uF-225-10-16V_C113841.html" H 4140 2730 50  0001 C CNN
 	1    4140 2730
 	1    0    0    -1
@@
 F 1 "475K  E96 series (tolerance 1%)" H 4350 3935 50  0000 L CNN
 F 2 "Resistors_SMD:R_0805_HandSoldering" V 4210 3980 50  0001 C CNN
-F 3 "~" H 4280 3980 50  0001 C CNN
+F 3 "RC0805FR-07475KL" H 4280 3980 50  0001 C CNN
 	1    4280 3980
 	1    0    0    -1
@@
 F 1 "402K E96 series (tolerance 1%)" H 4350 4325 50  0000 L CNN
 F 2 "Resistors_SMD:R_0805_HandSoldering" V 4210 4370 50  0001 C CNN
-F 3 "~" H 4280 4370 50  0001 C CNN
+F 3 "0805W8F4023T5E" H 4280 4370 50  0001 C CNN
 	1    4280 4370
 	1    0    0    -1
@@
 F 1 "HMHA2801" H 8630 4564 50  0000 C CNN
 F 2 "Housings_SSOP:SOP-4_4.4x2.8mm_Pitch1.27mm" H 8430 4130 50  0001 L CIN
-F 3 "https://uk.farnell.com/on-semiconductor/hmha2801/optocoupler-single-channel/dp/1652504" H 8630 4330 50  0001 L CNN
+F 3 "https://datasheet.lcsc.com/szlcsc/ON-Semicon-ON-HMHA2801_C232857.pdf" H 8630 4330 50  0001 L CNN
 	1    8630 4330
 	1    0    0    -1
@@
 F 1 "TX Connector" H 9353 4341 50  0000 R CNN
 F 2 "Connectors_JST:JST_PH_S2B-PH-K_02x2.00mm_Angled" H 9380 4370 50  0001 C CNN
-F 3 "~" H 9380 4370 50  0001 C CNN
+F 3 "https://datasheet.lcsc.com/szlcsc/JST-Sales-America-S2B-PH-K-S-LF-SN_C173752.pdf" H 9380 4370 50  0001 C CNN
 	1    9380 4370
 	-1   0    0    1
@@
 F 1 "510R" V 7954 4230 50  0000 C CNN
 F 2 "Resistors_SMD:R_0805_HandSoldering" V 8000 4230 50  0001 C CNN
-F 3 "~" H 8070 4230 50  0001 C CNN
+F 3 "RC0805FR-07510RL" H 8070 4230 50  0001 C CNN
 	1    8070 4230
 	0    1    1    0
@@
 F 1 "IRLML6244TRPBF" V 9121 2900 50  0000 C CNN
 F 2 "TO_SOT_Packages_SMD:SOT-23" H 8980 3000 50  0001 C CNN
-F 3 "https://lcsc.com/product-detail/MOSFET_Infineon-Technologies_IRLML6244TRPBF_Infineon-Technologies-IRLML6244TRPBF_C143946.html?promote=YjJhMTIxR3ZTWUlpbjVEZnUrY3Qvc09VOEYyOE14SkI2K0RRMVFoN2VDVURwMmNhNjVtZUR0Q0wyT2RYeHhqKzNieU5DVVdqZnBXTUFjSjU5ektWWlh3LzRDNXdTUGhOcWZHVEhWcnhuWjd5M1g0QzArUk1JMHppaGQ2QXgrZG9xc043STQvNw==" H 8780 2900 50  0001 C CNN
+F 3 "https://datasheet.lcsc.com/szlcsc/Infineon-Technologies-IRLML6244TRPBF_C143946.pdf" H 8780 2900 50  0001 C CNN
 	1    8780 2900
 	0    1    1    0
@@
 F 1 "47K" H 8300 2810 50  0000 L CNN
 F 2 "Resistors_SMD:R_0805_HandSoldering" V 8160 2850 50  0001 C CNN
-F 3 "YAGEO RC0805FR-0747KL" H 8230 2850 50  0001 C CNN
+F 3 "https://datasheet.lcsc.com/szlcsc/YAGEO-RC0805FR-0747KL_C126351.pdf" H 8230 2850 50  0001 C CNN
 	1    8230 2850
 	1    0    0    -1
@@
 F 1 "RX Connector" H 9203 5061 50  0000 R CNN
 F 2 "Connectors_JST:JST_PH_S2B-PH-K_02x2.00mm_Angled" H 9230 5090 50  0001 C CNN
-F 3 "http://www.farnell.com/datasheets/2057211.pdf" H 9230 5090 50  0001 C CNN
+F 3 "https://datasheet.lcsc.com/szlcsc/JST-Sales-America-S2B-PH-K-S-LF-SN_C173752.pdf" H 9230 5090 50  0001 C CNN
 	1    9230 5090
 	-1   0    0    1
@@
 F 1 "4K7" V 8474 5240 50  0000 C CNN
 F 2 "Resistors_SMD:R_0805_HandSoldering" V 8520 5240 50  0001 C CNN
-F 3 "~" H 8590 5240 50  0001 C CNN
+F 3 "RC0805FR-074K7L" H 8590 5240 50  0001 C CNN
 	1    8590 5240
 	-1   0    0    1
@@
 F 1 "RED LED" H 8070 1250 50  0000 C CNN
 F 2 "LEDs:LED_0805_HandSoldering" H 7980 1350 50  0001 C CNN
-F 3 "~" H 7980 1350 50  0001 C CNN
+F 3 "https://lcsc.com/product-detail/Light-Emitting-Diodes-LED_BL-HUF35A-AV-TRB-Iv-80mcd-Typ-atIF-20mA_C94741.html" H 7980 1350 50  0001 C CNN
 	1    7980 1350
 	-1   0    0    1
@@
 F 1 "2K2" V 8450 1230 50  0000 L CNN
 F 2 "Resistors_SMD:R_0805_HandSoldering" V 8290 1350 50  0001 C CNN
-F 3 "~" H 8360 1350 50  0001 C CNN
+F 3 "RC0805FR-072K2L" H 8360 1350 50  0001 C CNN
 	1    8360 1350
 	0    1    1    0
@@
 F 1 "Green" H 4340 3540 50  0000 C CNN
 F 2 "LEDs:LED_0805_HandSoldering" H 4310 3370 50  0001 C CNN
-F 3 "~" H 4310 3370 50  0001 C CNN
+F 3 "https://lcsc.com/product-detail/Light-Emitting-Diodes-LED_Emerald-SMDLED-Iv-220-270mcd-atIF-5mA_C84260.html" H 4310 3370 50  0001 C CNN
 	1    4310 3370
 	-1   0    0    1
@@
 F 1 "2K2" V 4780 3250 50  0000 L CNN
 F 2 "Resistors_SMD:R_0805_HandSoldering" V 4620 3370 50  0001 C CNN
-F 3 "~" H 4690 3370 50  0001 C CNN
+F 3 "RC0805FR-072K2L" H 4690 3370 50  0001 C CNN
 	1    4690 3370
 	0    1    1    0
@@
 F 1 "47K" H 2810 6935 50  0000 L CNN
 F 2 "Resistors_SMD:R_0805_HandSoldering" V 2670 6980 50  0001 C CNN
-F 3 "~" H 2740 6980 50  0001 C CNN
+F 3 "https://datasheet.lcsc.com/szlcsc/YAGEO-RC0805FR-0747KL_C126351.pdf" H 2740 6980 50  0001 C CNN
 	1    2740 6980
 	1    0    0    -1
@@
 F 1 "47K" H 4350 5995 50  0000 L CNN
 F 2 "Resistors_SMD:R_0805_HandSoldering" V 4210 6040 50  0001 C CNN
-F 3 "~" H 4280 6040 50  0001 C CNN
+F 3 "https://datasheet.lcsc.com/szlcsc/YAGEO-RC0805FR-0747KL_C126351.pdf" H 4280 6040 50  0001 C CNN
 	1    4280 6040
 	1    0    0    -1
@@
 F 1 "Remote temp input 47K @ 25oC" H 4850 5890 50  0000 R CNN
 F 2 "Pin_Headers:Pin_Header_Straight_1x05_Pitch2.54mm" H 4870 5650 50  0001 C CNN
-F 3 "~" H 4870 5650 50  0001 C CNN
+F 3 "https://lcsc.com/product-detail/Pin-Header-Female-Header_Shenzhen-Cankemeng-Headers-Pins-1-5P-2-54mm-Straight-line_C124379.html" H 4870 5650 50  0001 C CNN
 	1    4870 5650
 	-1   0    0    1
@@
 F 1 "510R" H 7450 2810 50  0000 L CNN
 F 2 "Resistors_SMD:R_0805_HandSoldering" V 7310 2870 50  0001 C CNN
-F 3 "" H 7380 2870 50  0001 C CNN
+F 3 "RC0805FR-07510RL" H 7380 2870 50  0001 C CNN
 	1    7380 2870
 	0    1    1    0
@@
 P 7670 1050
 F 0 "R22" V 7463 1050 50  0000 C CNN
-F 1 "4R4" V 7554 1050 50  0000 C CNN
+F 1 "10R" V 7554 1050 50  0000 C CNN
 F 2 "Resistors_THT:R_Axial_Power_L25.0mm_W9.0mm_P27.94mm" V 7600 1050 50  0001 C CNN
-F 3 "~" H 7670 1050 50  0001 C CNN
+F 3 "https://lcsc.com/product-detail/Others_Chian-Chia-Elec-CR-M5W-10RJ_C334310.html" H 7670 1050 50  0001 C CNN
 	1    7670 1050
 	0    1    1    0
@@
 $EndComp
 Text Notes 6640 760  0    50   ~ 0
-Either the SMD or larger power resistor is used - NOT BOTH!\n
+Either the SMD or larger power resistor is used - NOT BOTH !\nNote you must pick a resistor with correct power rating!
 Connection ~ 8510 1350
 Wire Wire Line
@@
 F 1 "Blue" H 4780 3100 50  0000 C CNN
 F 2 "LEDs:LED_0805" H 4750 2930 50  0001 C CNN
-F 3 "~" H 4750 2930 50  0001 C CNN
+F 3 "https://lcsc.com/product-detail/Light-Emitting-Diodes-LED_SMDLED-blue_C189307.html" H 4750 2930 50  0001 C CNN
 	1    4750 2930
 	-1   0    0    1
@@
 F 1 "2K2" V 5220 2810 50  0000 L CNN
 F 2 "Resistors_SMD:R_0805" V 5060 2930 50  0001 C CNN
-F 3 "~" H 5130 2930 50  0001 C CNN
+F 3 "RC0805FR-072K2L" H 5130 2930 50  0001 C CNN
 	1    5130 2930
 	0    1    1    0

Commit message: Reworked components in 0603 sizes for assembly in JLCPCB
Reworked components in 0603 sizes for assembly in JLCPCB and using standard parts list where possible
Parts:
- removed R22: 10R, Resistors_THT:R_Axial_Power_L25.0mm_W9.0mm_P27.94mm, symbol Device:R
- C1: footprint Capacitors_SMD:C_0805_HandSoldering -> Capacitors_SMD:C_0603; LCSCStockCode (none) -> C14663; PartNumber (none) -> CC0603KRX7R9BB104
- C2: footprint Capacitors_SMD:C_0805_HandSoldering -> Capacitors_SMD:C_0603; LCSCStockCode (none) -> C23630; PartNumber (none) -> CL10A225KO8NNNC
- C3: value 10uF 10V -> MLCC 10UF 10V; footprint Capacitors_SMD:C_0805_HandSoldering -> Capacitors_SMD:C_0603; LCSCStockCode (none) -> C19702; PartNumber (none) -> CL10A106KP8NNNC
- D2: footprint LEDs:LED_0805 -> LEDs:LED_0603; LCSCStockCode (none) -> C72041; PartNumber (none) -> 19-217/BHC-ZL1M2RY/3T
- D3: value RED LED -> Red; footprint LEDs:LED_0805_HandSoldering -> LEDs:LED_0603; LCSCStockCode (none) -> C2286; PartNumber (none) -> KT-0603R
- D4: footprint LEDs:LED_0805_HandSoldering -> LEDs:LED_0603; LCSCStockCode (none) -> C72043; PartNumber (none) -> 19-217/GHC-YR1S2/3T
- Q1: LCSCStockCode (none) -> C143946
- R1: footprint Resistors_SMD:R_0805_HandSoldering -> Resistors_SMD:R_0603; LCSCStockCode (none) -> C25804; PartNumber (none) -> 0603WAF1002T5E
- R10, R11, R12, R13, R6, R7, R8, R9: value 2R2 1W -> 2R 1W; LCSCStockCode (none) -> C49298; PartNumber (none) -> 25121WF200KT4E
- R14, R5: footprint Resistors_SMD:R_0805_HandSoldering -> Resistors_SMD:R_0603; LCSCStockCode (none) -> C23193; PartNumber (none) -> 0603WAF5100T5E
- R15, R20, R21: footprint Resistors_SMD:R_0805_HandSoldering -> Resistors_SMD:R_0603; LCSCStockCode (none) -> C25819; PartNumber (none) -> 0603WAF4702T5E
- R16: footprint Resistors_SMD:R_0805_HandSoldering -> Resistors_SMD:R_0603; LCSCStockCode (none) -> C23162; PartNumber (none) -> 0603WAF4701T5E
- R17, R18: footprint Resistors_SMD:R_0805_HandSoldering -> Resistors_SMD:R_0603; LCSCStockCode (none) -> C4190; PartNumber (none) -> 0603WAF2201T5E
- R19: value SDNT2012X473F4150FTF -> NCP18WB473J03RB; footprint Resistors_SMD:R_0805_HandSoldering -> Resistors_SMD:R_0603; LCSCStockCode (none) -> C86142; PartNumber (none) -> NCP18WB473J03RB
- R2: footprint Resistors_SMD:R_0805_HandSoldering -> Resistors_SMD:R_0603; LCSCStockCode (none) -> C21190; PartNumber (none) -> 0603WAF1001T5E
- R23: footprint Resistors_SMD:R_0805 -> Resistors_SMD:R_0603; LCSCStockCode (none) -> C4190; PartNumber (none) -> 0603WAF2201T5E
- R3: value 475K E96 series (tolerance 1%) -> 475K E96 series (tolerance 1%); footprint Resistors_SMD:R_0805_HandSoldering -> Resistors_SMD:R_0603; LCSCStockCode (none) -> C23180; PartNumber (none) -> 0603WAF4753T5E
- R4: footprint Resistors_SMD:R_0805_HandSoldering -> Resistors_SMD:R_0603; LCSCStockCode (none) -> C23048; PartNumber (none) -> 0603WAF4023T5E
- U1: LCSCStockCode (none) -> C232857
- U4: LCSCStockCode (none) -> C219103
Connections:
- wire segments 131 -> 128
Other:
- note added: "Each row is 8R and 4W max (needs to carry 2.2W @ 4.2V), drops about 525mA.\n"
- note removed: "Each row is 8R8 and 4W max (needs to carry 2W @ 4.2V), drops about 470mA.\n"
- note removed: "Ever Ohms Tech CR2512F2R2E04\nhttps://lcsc.com/product-detail/Chip-Resistor-Surface-Mount_Ever-Ohms-Tech-CR2512F2R2E04_C147074.html\n"

Commit message: Minor tweaks to LED brightness
Parts:
- D1: value LM4040BIM3-2.0/NOPB, 2.048V, SOT-23-3 -> LM4040A20IDBZR 2.048V, SOT-23-3; LCSCStockCode (none) -> C127070; PartNumber (none) -> LM4040A20IDBZR
- R23: value 2K2 -> 1K8; LCSCStockCode C4190 -> C4177; PartNumber 0603WAF2201T5E -> 0603WAF1801T5E
- U1: value HMHA2801 -> HMHA2801AR2; LCSCStockCode C232857 -> C258257
Changed lines of the file:
@@
 P 3360 2760
 F 0 "D1" V 3406 2672 50  0000 R CNN
-F 1 "LM4040BIM3-2.0/NOPB, 2.048V, SOT-23-3" V 3620 2390 50  0000 R CNN
+F 1 "LM4040A20IDBZR 2.048V, SOT-23-3" V 3600 2720 50  0000 R CNN
 F 2 "TO_SOT_Packages_SMD:SOT-23" H 3360 2560 50  0001 C CIN
 F 3 "https://uk.farnell.com/texas-instruments/lm4040bim3-2-0-nopb/voltage-ref-shunt-2-048v-sot-23/dp/2492201" H 3360 2760 50  0001 C CIN
+F 4 "C127070" V 3360 2760 50  0001 C CNN "LCSCStockCode"
+F 5 "LM4040A20IDBZR" V 3360 2760 50  0001 C CNN "PartNumber"
 	1    3360 2760
 	0    -1   -1   0
@@
 P 8630 4330
 F 0 "U1" H 8630 4655 50  0000 C CNN
-F 1 "HMHA2801" H 8630 4564 50  0000 C CNN
+F 1 "HMHA2801AR2" H 8630 4564 50  0000 C CNN
 F 2 "Housings_SSOP:SOP-4_4.4x2.8mm_Pitch1.27mm" H 8430 4130 50  0001 L CIN
-F 3 "https://datasheet.lcsc.com/szlcsc/ON-Semicon-ON-HMHA2801_C232857.pdf" H 8630 4330 50  0001 L CNN
-F 4 "C232857" H 8630 4330 50  0001 C CNN "LCSCStockCode"
+F 3 "" H 8630 4330 50  0001 L CNN
+F 4 "C258257" H 8630 4330 50  0001 C CNN "LCSCStockCode"
 	1    8630 4330
 	1    0    0    -1
@@
 P 5130 2930
 F 0 "R23" V 5220 2980 50  0000 L CNN
-F 1 "2K2" V 5220 2810 50  0000 L CNN
+F 1 "1K8" V 5220 2810 50  0000 L CNN
 F 2 "Resistors_SMD:R_0603" V 5060 2930 50  0001 C CNN
 F 3 "" H 5130 2930 50  0001 C CNN
-F 4 "C4190" V 2560 4410 50  0001 C CNN "LCSCStockCode"
-F 5 "0603WAF2201T5E" V 2560 4410 50  0001 C CNN "PartNumber"
+F 4 "C4177" V 2560 4410 50  0001 C CNN "LCSCStockCode"
+F 5 "0603WAF1801T5E" V 2560 4410 50  0001 C CNN "PartNumber"
 	1    5130 2930
 	0    1    1    0
