File: Circuit/v4.sch (KiCad schematic (older format))
At the start: 37 parts, among them J2 AVR-ISP-6, Q1 IRLML6244TRPBF, U1 HMHA2801AR2, U4 ATtiny841-SSU

Commit message: Updated Gerber - doesnt work dont use
Parts:
- D1: value LM4040A20IDBZR 2.048V, SOT-23-3 -> Fixed 2.048V; LCSCStockCode C127070 -> C48833; PartNumber LM4040A20IDBZR -> ADR5040BRTZ-REEL7
Changed lines of the file:
@@
 P 3360 2760
 F 0 "D1" V 3406 2672 50  0000 R CNN
-F 1 "LM4040A20IDBZR 2.048V, SOT-23-3" V 3600 2720 50  0000 R CNN
+F 1 "Fixed 2.048V" V 3600 2720 50  0000 R CNN
 F 2 "TO_SOT_Packages_SMD:SOT-23" H 3360 2560 50  0001 C CIN
-F 3 "https://uk.farnell.com/texas-instruments/lm4040bim3-2-0-nopb/voltage-ref-shunt-2-048v-sot-23/dp/2492201" H 3360 2760 50  0001 C CIN
-F 4 "C127070" V 3360 2760 50  0001 C CNN "LCSCStockCode"
-F 5 "LM4040A20IDBZR" V 3360 2760 50  0001 C CNN "PartNumber"
+F 3 "" H 3360 2760 50  0001 C CIN
+F 4 "C48833" V 3360 2760 50  0001 C CNN "LCSCStockCode"
+F 5 "ADR5040BRTZ-REEL7" V 3360 2760 50  0001 C CNN "PartNumber"
 	1    3360 2760
 	0    -1   -1   0

Commit message: Correct layout for JLCPCB - prototype parts
This design contains UNTESTED components (ADZ5040 and HMHA2801A) build at your own risk/cost
Parts:
- D1: value Fixed 2.048V -> ADR5040BRTZ-REEL7 2.048V
Changed lines of the file:
@@
 P 3360 2760
 F 0 "D1" V 3406 2672 50  0000 R CNN
-F 1 "Fixed 2.048V" V 3600 2720 50  0000 R CNN
+F 1 "ADR5040BRTZ-REEL7 2.048V" V 3600 2720 50  0000 R CNN
 F 2 "TO_SOT_Packages_SMD:SOT-23" H 3360 2560 50  0001 C CIN
-F 3 "" H 3360 2760 50  0001 C CIN
+F 3 "https://datasheet.lcsc.com/szlcsc/1810161810_Analog-Devices-ADR5040BRTZ-REEL7_C48833.pdf" H 3360 2760 50  0001 C CIN
 F 4 "C48833" V 3360 2760 50  0001 C CNN "LCSCStockCode"
 F 5 "ADR5040BRTZ-REEL7" V 3360 2760 50  0001 C CNN "PartNumber"

Commit message: Change resistors in voltage divider to JLCPCB basic parts to reduce cost
Parts:
- R3: value 475K E96 series (tolerance 1%) -> 470KOHMS ±1% 1/10W; LCSCStockCode C23180 -> C23178; PartNumber 0603WAF4753T5E -> 0603WAF4703T5E
- R4: value 402K E96 series (tolerance 1%) -> 390KOHMS ±1% 1/10W; LCSCStockCode C23048 -> C23150; PartNumber 0603WAF4023T5E -> 0603WAF3903T5E
Other:
- note added: "Output voltage 2.048 for input of 4.516V (max)"
- note removed: "Output voltage 2.048 for input of 4.468V (max)"
Changed lines of the file:
@@
 P 4280 3980
 F 0 "R3" H 4350 4026 50  0000 L CNN
-F 1 "475K E96 series (tolerance 1%)" H 4350 3935 50  0000 L CNN
+F 1 "470KOHMS ±1% 1/10W" H 4350 3935 50  0000 L CNN
 F 2 "Resistors_SMD:R_0603" V 4210 3980 50  0001 C CNN
 F 3 "" H 4280 3980 50  0001 C CNN
-F 4 "C23180" V 2560 4410 50  0001 C CNN "LCSCStockCode"
-F 5 "0603WAF4753T5E" V 2560 4410 50  0001 C CNN "PartNumber"
+F 4 "C23178" V 2560 4410 50  0001 C CNN "LCSCStockCode"
+F 5 "0603WAF4703T5E" V 2560 4410 50  0001 C CNN "PartNumber"
 	1    4280 3980
 	1    0    0    -1
@@
 P 4280 4370
 F 0 "R4" H 4350 4416 50  0000 L CNN
-F 1 "402K E96 series (tolerance 1%)" H 4350 4325 50  0000 L CNN
+F 1 "390KOHMS ±1% 1/10W" H 4350 4325 50  0000 L CNN
 F 2 "Resistors_SMD:R_0603" V 4210 4370 50  0001 C CNN
 F 3 "" H 4280 4370 50  0001 C CNN
-F 4 "C23048" V 2560 4410 50  0001 C CNN "LCSCStockCode"
-F 5 "0603WAF4023T5E" V 2560 4410 50  0001 C CNN "PartNumber"
+F 4 "C23150" V 2560 4410 50  0001 C CNN "LCSCStockCode"
+F 5 "0603WAF3903T5E" V 2560 4410 50  0001 C CNN "PartNumber"
 	1    4280 4370
 	1    0    0    -1
@@
 	2250 3770 2430 3770
 Text Notes 4760 4250 0    50   ~ 0
-Output voltage 2.048 for input of 4.468V (max)
+Output voltage 2.048 for input of 4.516V (max)
 Text Notes 3640 2230 0    50   ~ 0
 AREF input acts like a resistor of 32k from AREF to GND

Commit message: Version 4.2 complete
Parts:
- renumbered U4 to ATTINY841
Changed lines of the file:
@@
 $EndDescr
 $Comp
-L v4-rescue:ATtiny841-SSU-MCU_Microchip_ATtiny-v4-rescue U4
+L v4-rescue:ATtiny841-SSU-MCU_Microchip_ATtiny-v4-rescue ATTINY841
 U 1 1 5BC63D51
 P 1650 3670
-F 0 "U4" H 1120 3716 50  0000 R CNN
+F 0 "ATTINY841" H 1120 3716 50  0000 R CNN
 F 1 "ATtiny841-SSU" H 1120 3625 50  0000 R CNN
 F 2 "Housings_SOIC:SOIC-14_3.9x8.7mm_Pitch1.27mm" H 1650 3670 50  0001 C CIN

Commit message: Redesigned circuit using TCLT1003 optoisolator
For 30 boards
Charge Details
Engineering fee:$4.00
Board:$3.10
SMT Price:
Setup fee:$7.00
Stencil:$0.00
Panel:$0.00
Components:$37.27
Extended components fee:$15.00
Total Price:$66.37
Parts:
- U1: value HMHA2801AR2 -> TCLT1003; footprint Housings_SSOP:SOP-4_4.4x2.8mm_Pitch1.27mm -> Circuit:SOP4-L-Pitch2.54; LCSCStockCode C258257 -> C118296; PartNumber (none) -> TCLT1003
Other:
- note added: "Optocoupler, Phototransistor Output,\nSOP-4L, Long Mini-Flat Package\n"
- note removed: "Optocoupler, Phototransistor Output,\n4-SSOP"
Changed lines of the file:
@@
 P 8630 4330
 F 0 "U1" H 8630 4655 50  0000 C CNN
-F 1 "HMHA2801AR2" H 8630 4564 50  0000 C CNN
-F 2 "Housings_SSOP:SOP-4_4.4x2.8mm_Pitch1.27mm" H 8430 4130 50  0001 L CIN
-F 3 "" H 8630 4330 50  0001 L CNN
-F 4 "C258257" H 8630 4330 50  0001 C CNN "LCSCStockCode"
+F 1 "TCLT1003" H 8630 4564 50  0000 C CNN
+F 2 "Circuit:SOP4-L-Pitch2.54" H 8430 4130 50  0001 L CIN
+F 3 "https://datasheet.lcsc.com/szlcsc/Vishay-Intertech-TCLT1003_C118296.pdf" H 8630 4330 50  0001 L CNN
+F 4 "C118296" H 8630 4330 50  0001 C CNN "LCSCStockCode"
+F 5 "TCLT1003" H 8630 4330 50  0001 C CNN "PartNumber"
 	1    8630 4330
 	1    0    0    -1
@@
 ENABLE
 Text Notes 8150 3920 0    50   ~ 0
-Optocoupler, Phototransistor Output,\n4-SSOP
+Optocoupler, Phototransistor Output,\nSOP-4L, Long Mini-Flat Package\n
 Wire Wire Line
 	2250 3070 3020 3070

Commit message: Updated Green LED to match JLCPCB parts list
Parts:
- D4: LCSCStockCode C72043 -> C72042; PartNumber 19-217/GHC-YR1S2/3T -> 19-217/G7C-AN1P2/3T
Changed lines of the file:
@@
 F 1 "Green" H 4340 3540 50  0000 C CNN
 F 2 "LEDs:LED_0603" H 4310 3370 50  0001 C CNN
-F 3 "" H 4310 3370 50  0001 C CNN
-F 4 "C72043" H 4310 3370 50  0001 C CNN "LCSCStockCode"
-F 5 "19-217/GHC-YR1S2/3T" H 4310 3370 50  0001 C CNN "PartNumber"
+F 3 "https://datasheet.lcsc.com/szlcsc/Everlight-Elec-19-217-G7C-AN1P2-3T_C72042.pdf" H 4310 3370 50  0001 C CNN
+F 4 "C72042" H 4310 3370 50  0001 C CNN "LCSCStockCode"
+F 5 "19-217/G7C-AN1P2/3T" H 4310 3370 50  0001 C CNN "PartNumber"
 	1    4310 3370
 	-1   0    0    1

Commit message: Change components to reduce cost against JLCPCB parts
Parts:
- D4: footprint LEDs:LED_0603 -> LEDs:LED_0805; LCSCStockCode C72042 -> C2297; PartNumber 19-217/G7C-AN1P2/3T -> Hubei KENTO Elec Green 0805
- U1: value TCLT1003 -> EL3H7(B)(TA)-G; footprint Circuit:SOP4-L-Pitch2.54 -> Housings_SSOP:SOP-4_4.4x2.8mm_Pitch1.27mm; LCSCStockCode C118296 -> C32565; PartNumber TCLT1003 -> EL3H7(B)(TA)-G
Other:
- note added: "4 PIN ULTRA SMALL SSOP\nPHOTOTRANSISTOR PHOTOCOUPLER EL3H7-G Series\n"
- note added: "Each row is 8R and 4W max. Needs to carry 4.41W total @ 4.2V max 1050mA.\n"
- note removed: "Each row is 8R and 4W max (needs to carry 2.2W @ 4.2V), drops about 525mA.\n"
- note removed: "Either the SMD or larger power resistor is used - NOT BOTH !\nNote you must pick a resistor with correct power rating!"
- note removed: "Optocoupler, Phototransistor Output,\nSOP-4L, Long Mini-Flat Package\n"
Changed lines of the file:
@@
 P 8630 4330
 F 0 "U1" H 8630 4655 50  0000 C CNN
-F 1 "TCLT1003" H 8630 4564 50  0000 C CNN
-F 2 "Circuit:SOP4-L-Pitch2.54" H 8430 4130 50  0001 L CIN
-F 3 "https://datasheet.lcsc.com/szlcsc/Vishay-Intertech-TCLT1003_C118296.pdf" H 8630 4330 50  0001 L CNN
-F 4 "C118296" H 8630 4330 50  0001 C CNN "LCSCStockCode"
-F 5 "TCLT1003" H 8630 4330 50  0001 C CNN "PartNumber"
+F 1 "EL3H7(B)(TA)-G" H 8630 4564 50  0000 C CNN
+F 2 "Housings_SSOP:SOP-4_4.4x2.8mm_Pitch1.27mm" H 8430 4130 50  0001 L CIN
+F 3 "https://datasheet.lcsc.com/szlcsc/Everlight-Elec-EL3H7-B-TA-G_C32565.pdf" H 8630 4330 50  0001 L CNN
+F 4 "C32565" H 8630 4330 50  0001 C CNN "LCSCStockCode"
+F 5 "EL3H7(B)(TA)-G" H 8630 4330 50  0001 C CNN "PartNumber"
 	1    8630 4330
 	1    0    0    -1
@@
 	8050 1990 8100 1990
 Text Notes 5990 1620 0    50   ~ 0
-Each row is 8R and 4W max (needs to carry 2.2W @ 4.2V), drops about 525mA.\n
+Each row is 8R and 4W max. Needs to carry 4.41W total @ 4.2V max 1050mA.\n
 $Comp
 L Device:R R7
@@
 F 0 "D4" H 4450 3470 50  0000 C CNN
 F 1 "Green" H 4340 3540 50  0000 C CNN
-F 2 "LEDs:LED_0603" H 4310 3370 50  0001 C CNN
-F 3 "https://datasheet.lcsc.com/szlcsc/Everlight-Elec-19-217-G7C-AN1P2-3T_C72042.pdf" H 4310 3370 50  0001 C CNN
-F 4 "C72042" H 4310 3370 50  0001 C CNN "LCSCStockCode"
-F 5 "19-217/G7C-AN1P2/3T" H 4310 3370 50  0001 C CNN "PartNumber"
+F 2 "LEDs:LED_0805" H 4310 3370 50  0001 C CNN
+F 3 "https://datasheet.lcsc.com/szlcsc/Hubei-KENTO-Elec-Green-0805-Iv-207-249-mcd-atIF-20mA_C2297.pdf" H 4310 3370 50  0001 C CNN
+F 4 "C2297" H 4310 3370 50  0001 C CNN "LCSCStockCode"
+F 5 "Hubei KENTO Elec Green 0805" H 4310 3370 50  0001 C CNN "PartNumber"
 	1    4310 3370
 	-1   0    0    1
@@
 Text GLabel 4560 5550 0    50   Input ~ 0
 ENABLE
-Text Notes 8150 3920 0    50   ~ 0
-Optocoupler, Phototransistor Output,\nSOP-4L, Long Mini-Flat Package\n
+Text Notes 7880 3940 0    50   ~ 0
+4 PIN ULTRA SMALL SSOP\nPHOTOTRANSISTOR PHOTOCOUPLER EL3H7-G Series\n
 Wire Wire Line
 	2250 3070 3020 3070
@@
 	1    0    0    -1
 $EndComp
-Text Notes 6640 760  0    50   ~ 0
-Either the SMD or larger power resistor is used - NOT BOTH !\nNote you must pick a resistor with correct power rating!
 Wire Wire Line
 	7540 1350 7540 1050

Commit message: Changes to parts to keep on JLC basic list and reduce cost
Parts:
- C1: footprint Capacitors_SMD:C_0603 -> Capacitors_SMD:C_0805; LCSCStockCode C14663 -> C49678; PartNumber CC0603KRX7R9BB104 -> CC0805KRX7R9BB104
- D2: footprint LEDs:LED_0603 -> LEDs:LED_0805; LCSCStockCode C72041 -> C2293; PartNumber 19-217/BHC-ZL1M2RY/3T -> HUBEI KENTO ELEC
- D3: footprint LEDs:LED_0603 -> LEDs:LED_0805; LCSCStockCode C2286 -> C84256; PartNumber KT-0603R -> FC-2012HRK-620D
- R3: value 470KOHMS ±1% 1/10W -> 470KOHMS 1% 1/10W
- R4: value 390KOHMS ±1% 1/10W -> 390KOHMS 1% 1/10W
Changed lines of the file:
@@
 F 0 "C1" H 836 2926 50  0000 R CNN
 F 1 "100nF" H 836 2835 50  0000 R CNN
-F 2 "Capacitors_SMD:C_0603" H 988 2730 50  0001 C CNN
+F 2 "Capacitors_SMD:C_0805" H 988 2730 50  0001 C CNN
 F 3 "" H 950 2880 50  0001 C CNN
-F 4 "C14663" H 950 2880 50  0001 C CNN "LCSCStockCode"
-F 5 "CC0603KRX7R9BB104" H 950 2880 50  0001 C CNN "PartNumber"
+F 4 "C49678" H 950 2880 50  0001 C CNN "LCSCStockCode"
+F 5 "CC0805KRX7R9BB104" H 950 2880 50  0001 C CNN "PartNumber"
 	1    950  2880
 	1    0    0    -1
@@
 P 4280 3980
 F 0 "R3" H 4350 4026 50  0000 L CNN
-F 1 "470KOHMS ±1% 1/10W" H 4350 3935 50  0000 L CNN
+F 1 "470KOHMS 1% 1/10W" H 4350 3935 50  0000 L CNN
 F 2 "Resistors_SMD:R_0603" V 4210 3980 50  0001 C CNN
 F 3 "" H 4280 3980 50  0001 C CNN
@@
 P 4280 4370
 F 0 "R4" H 4350 4416 50  0000 L CNN
-F 1 "390KOHMS ±1% 1/10W" H 4350 4325 50  0000 L CNN
+F 1 "390KOHMS 1% 1/10W" H 4350 4325 50  0000 L CNN
 F 2 "Resistors_SMD:R_0603" V 4210 4370 50  0001 C CNN
 F 3 "" H 4280 4370 50  0001 C CNN
@@
 F 0 "D3" H 8120 1450 50  0000 C CNN
 F 1 "Red" H 8070 1250 50  0000 C CNN
-F 2 "LEDs:LED_0603" H 7980 1350 50  0001 C CNN
+F 2 "LEDs:LED_0805" H 7980 1350 50  0001 C CNN
 F 3 "" H 7980 1350 50  0001 C CNN
-F 4 "C2286" H 7980 1350 50  0001 C CNN "LCSCStockCode"
-F 5 "KT-0603R" H 7980 1350 50  0001 C CNN "PartNumber"
+F 4 "C84256" H 7980 1350 50  0001 C CNN "LCSCStockCode"
+F 5 "FC-2012HRK-620D" H 7980 1350 50  0001 C CNN "PartNumber"
 	1    7980 1350
 	-1   0    0    1
@@
 F 0 "D2" H 4890 3030 50  0000 C CNN
 F 1 "Blue" H 4780 3100 50  0000 C CNN
-F 2 "LEDs:LED_0603" H 4750 2930 50  0001 C CNN
+F 2 "LEDs:LED_0805" H 4750 2930 50  0001 C CNN
 F 3 "" H 4750 2930 50  0001 C CNN
-F 4 "C72041" H 4750 2930 50  0001 C CNN "LCSCStockCode"
-F 5 "19-217/BHC-ZL1M2RY/3T" H 4750 2930 50  0001 C CNN "PartNumber"
+F 4 "C2293" H 4750 2930 50  0001 C CNN "LCSCStockCode"
+F 5 "HUBEI KENTO ELEC" H 4750 2930 50  0001 C CNN "PartNumber"
 	1    4750 2930
 	-1   0    0    1
