File: ESP8266ControllerCircuit/ESP8266ControllerCircuit.sch (KiCad schematic (older format))
At the start: 20 parts, among them J1 Input, J2 Input, J3 Input, J4 Input, J5 Optional, U1 WeMos_mini, U2 HMHA2801, U3 PCF8574T/3,518

Commit message: Rename of ESP to ESP8266
Parts:
- U1: footprint ESPControllerCircuit:wemos-d1-mini-with-pin-header -> ESP8266ControllerCircuit:wemos-d1-mini-with-pin-header
Changed lines of the file:
@@
 encoding utf-8
 Sheet 1 1
-Title ""
-Date ""
-Rev ""
-Comp ""
-Comment1 ""
+Title "diyBMS ESP8266 Controller [legacy]"
+Date "2021-03-08"
+Rev "ESP8266"
+Comp "Stuart Pittaway"
+Comment1 "NOT FOR NEW DESIGNS"
 Comment2 ""
 Comment3 ""
@@
 F 0 "U1" H 2640 7117 60  0000 C CNN
 F 1 "WeMos_mini" H 2640 7011 60  0000 C CNN
-F 2 "ESPControllerCircuit:wemos-d1-mini-with-pin-header" H 3190 5780 60  0001 C CNN
+F 2 "ESP8266ControllerCircuit:wemos-d1-mini-with-pin-header" H 3190 5780 60  0001 C CNN
 F 3 "" H 3190 5780 60  0000 C CNN
 	1    2640 6480

Commit message: Updated ESP8266 controller BOM and Gerber
Parts:
- D1: footprint LEDs:LED_D5.0mm -> LEDs:LED_0805; LCSCStockCode (none) -> C2297; PartNumber (none) -> Hubei KENTO Elec Green 0805
- R1: LCSCStockCode (none) -> C17710; PartNumber (none) -> 0805W8F4700T5E
- R2: LCSCStockCode (none) -> C17520; PartNumber (none) -> 0805W8F2201T5E
- R3: LCSCStockCode (none) -> C17557; PartNumber (none) -> 0805W8F2200T5E
- R4, R5: LCSCStockCode (none) -> C17673; PartNumber (none) -> 0805W8F4701T5E
- U2: value HMHA2801 -> EL3H7(B)(TA)-G; LCSCStockCode (none) -> C32565
- U3: footprint SMD_Packages:SO-16-W -> Housings_SOIC:SOIC-16W_7.5x10.3mm_Pitch1.27mm; LCSCStockCode (none) -> C7605; PartNumber (none) -> PCF8574T/3,518
Connections:
- no-connect marks 3 -> 0
Changed lines of the file:
@@
 F 0 "D1" H 4040 6540 50  0000 C CNN
 F 1 "COMMS" H 4030 6720 50  0000 C CNN
-F 2 "LEDs:LED_D5.0mm" H 4040 6630 50  0001 C CNN
-F 3 "~" H 4040 6630 50  0001 C CNN
+F 2 "LEDs:LED_0805" H 4040 6630 50  0001 C CNN
+F 3 "https://datasheet.lcsc.com/szlcsc/Hubei-KENTO-Elec-Green-0805-Iv-207-249-mcd-atIF-20mA_C2297.pdf" H 4040 6630 50  0001 C CNN
+F 4 "C2297" H 4040 6630 50  0001 C CNN "LCSCStockCode"
+F 5 "Hubei KENTO Elec Green 0805" H 4040 6630 50  0001 C CNN "PartNumber"
 	1    4040 6630
 	-1   0    0    1
@@
 F 2 "Resistors_SMD:R_0805_HandSoldering" V 3510 6630 50  0001 C CNN
 F 3 "~" H 3580 6630 50  0001 C CNN
+F 4 "C17710" H 3580 6630 50  0001 C CNN "LCSCStockCode"
+F 5 "0805W8F4700T5E" H 3580 6630 50  0001 C CNN "PartNumber"
 	1    3580 6630
 	0    1    1    0
@@
 P 3960 5110
 F 0 "U2" H 3960 5435 50  0000 C CNN
-F 1 "HMHA2801" H 3960 5344 50  0000 C CNN
+F 1 "EL3H7(B)(TA)-G" H 3960 5344 50  0000 C CNN
 F 2 "Housings_SSOP:SOP-4_4.4x2.8mm_Pitch1.27mm" H 3760 4910 50  0001 L CIN
-F 3 "https://uk.farnell.com/on-semiconductor/hmha2801/optocoupler-single-channel/dp/1652504" H 3960 5110 50  0001 L CNN
+F 3 "https://datasheet.lcsc.com/szlcsc/Everlight-Elec-EL3H7-B-TA-G_C32565.pdf" H 3960 5110 50  0001 L CNN
+F 4 "C32565" H 3960 5110 50  0001 C CNN "LCSCStockCode"
 	1    3960 5110
 	1    0    0    -1
@@
 F 2 "Resistors_SMD:R_0805_HandSoldering" V 3860 5790 50  0001 C CNN
 F 3 "~" H 3930 5790 50  0001 C CNN
+F 4 "C17520" H 3930 5790 50  0001 C CNN "LCSCStockCode"
+F 5 "0805W8F2201T5E" H 3930 5790 50  0001 C CNN "PartNumber"
 	1    3930 5790
 	-1   0    0    1
@@
 F 2 "Resistors_SMD:R_0805_HandSoldering" V 3370 5010 50  0001 C CNN
 F 3 "~" H 3440 5010 50  0001 C CNN
+F 4 "C17557" V 3440 5010 50  0001 C CNN "LCSCStockCode"
+F 5 "0805W8F2200T5E" V 3440 5010 50  0001 C CNN "PartNumber"
 	1    3440 5010
 	0    1    1    0
@@
 F 2 "Resistors_SMD:R_0805_HandSoldering" V 1760 3350 50  0001 C CNN
 F 3 "~" H 1830 3350 50  0001 C CNN
+F 4 "C17673" H 1830 3350 50  0001 C CNN "LCSCStockCode"
+F 5 "0805W8F4701T5E" H 1830 3350 50  0001 C CNN "PartNumber"
 	1    1830 3350
 	1    0    0    -1
@@
 F 2 "Resistors_SMD:R_0805_HandSoldering" V 1950 3350 50  0001 C CNN
 F 3 "~" H 2020 3350 50  0001 C CNN
+F 4 "C17673" H 2020 3350 50  0001 C CNN "LCSCStockCode"
+F 5 "0805W8F4701T5E" H 2020 3350 50  0001 C CNN "PartNumber"
 	1    2020 3350
 	1    0    0    -1
@@
 F 0 "U3" H 2670 4781 50  0000 C CNN
 F 1 "PCF8574T/3,518" H 2690 4880 50  0000 C CNN
-F 2 "SMD_Packages:SO-16-W" H 2670 3900 50  0001 C CNN
+F 2 "Housings_SOIC:SOIC-16W_7.5x10.3mm_Pitch1.27mm" H 2670 3900 50  0001 C CNN
 F 3 "https://lcsc.com/product-detail/I-O-Expansion_NXP_PCF8574T-3-518_PCF8574T-3-518_C7605.html" H 2670 3900 50  0001 C CNN
+F 4 "" H 2670 3900 50  0001 C CNN "LCSCPart"
+F 5 "C7605" H 2670 3900 50  0001 C CNN "LCSCStockCode"
+F 6 "PCF8574T/3,518" H 2670 3900 50  0001 C CNN "PartNumber"
 	1    2670 3900
 	1    0    0    -1
@@
 Text Notes 5150 4430 0    50   ~ 0
 J1-J4 switch inputs (not optoisolated!)
+Wire Wire Line
+	3140 6430 3420 6430
+Wire Wire Line
+	3420 6430 3420 6290
+Wire Wire Line
+	3420 6290 4670 6290
+Wire Wire Line
+	4670 6290 4670 6410
+Wire Wire Line
+	4670 6410 4920 6410
+$Comp
+L power:GND #PWR05
+U 1 1 5CEE7CB3
+P 4620 6050
+F 0 "#PWR05" H 4620 5800 50  0001 C CNN
+F 1 "GND" H 4625 5877 50  0000 C CNN
+F 2 "" H 4620 6050 50  0001 C CNN
+F 3 "" H 4620 6050 50  0001 C CNN
+	1    4620 6050
+	1    0    0    -1
+$EndComp
+$Comp
+L power:+3.3V #PWR06
+U 1 1 5CEE831F
+P 4900 6050
+F 0 "#PWR06" H 4900 5900 50  0001 C CNN
+F 1 "+3.3V" H 4915 6223 50  0000 C CNN
+F 2 "" H 4900 6050 50  0001 C CNN
+F 3 "" H 4900 6050 50  0001 C CNN
+	1    4900 6050
+	1    0    0    -1
+$EndComp
+Wire Wire Line
+	4900 6050 4900 6210
+Wire Wire Line
+	4900 6210 4920 6210
+Wire Wire Line
+	4920 6310 4750 6310
+Wire Wire Line
+	4750 6310 4750 6050
+Wire Wire Line
+	4750 6050 4620 6050
 $Comp
 L Connector:Conn_01x03_Male J5
@@
 	-1   0    0    1
 $EndComp
-Wire Wire Line
-	3140 6430 3420 6430
-Wire Wire Line
-	3420 6430 3420 6290
-Wire Wire Line
-	3420 6290 4670 6290
-Wire Wire Line
-	4670 6290 4670 6410
-Wire Wire Line
-	4670 6410 4920 6410
-$Comp
-L power:GND #PWR05
-U 1 1 5CEE7CB3
-P 4620 6050
-F 0 "#PWR05" H 4620 5800 50  0001 C CNN
-F 1 "GND" H 4625 5877 50  0000 C CNN
-F 2 "" H 4620 6050 50  0001 C CNN
-F 3 "" H 4620 6050 50  0001 C CNN
-	1    4620 6050
-	1    0    0    -1
-$EndComp
-$Comp
-L power:+3.3V #PWR06
-U 1 1 5CEE831F
-P 4900 6050
-F 0 "#PWR06" H 4900 5900 50  0001 C CNN
-F 1 "+3.3V" H 4915 6223 50  0000 C CNN
-F 2 "" H 4900 6050 50  0001 C CNN
-F 3 "" H 4900 6050 50  0001 C CNN
-	1    4900 6050
-	1    0    0    -1
-$EndComp
-Wire Wire Line
-	4900 6050 4900 6210
-Wire Wire Line
-	4900 6210 4920 6210
-Wire Wire Line
-	4920 6310 4750 6310
-Wire Wire Line
-	4750 6310 4750 6050
-Wire Wire Line
-	4750 6050 4620 6050
-NoConn ~ 2140 6730
-NoConn ~ 2140 6830
-NoConn ~ 3140 6830
 $EndSCHEMATC
