File: ModuleV450/ModuleV450.kicad_pcb (KiCad board)
At the start: 2 copper layers, 30 x 61.3 mm, 43 parts, among them J1 J, J2 Comms, Q1 AO3400A, U1 EL3H7(B)(TA)-G, U2 ATTINY1624-SSU-ND

Commit message: Minor silkscreen changes
Parts:
- moved UPDI1 0.29 mm to (105.0, 64.7)
Other:
- board text added: "D"
- board text removed: "A"

Commit message: Temp sensor snap off board
Parts:
- added REF**: H1, Mounting_Holes:MountingHole_3.2mm_M3, F.Cu at (107.2, 100.1)
- added REF**: H1, Mounting_Holes:MountingHole_3.2mm_M3, F.Cu at (106.4, 100.1)
- added REF**: H1, Mounting_Holes:MountingHole_3.2mm_M3, F.Cu at (105.6, 100.1)
- added REF**: H1, Mounting_Holes:MountingHole_3.2mm_M3, F.Cu at (104.8, 100.1)
- moved J1 0.95 mm to (109.1, 103.1)
Routing:
- net ENABLE: track 85.5 -> 86.4 mm
- net PA3: track 58.8 -> 59.3 mm
Other:
- outline, holes or cut-outs redrawn
