File: ModuleV490-AllInOne/PowerSupply.kicad_sch (KiCad schematic)
At the start: 28 parts, among them J5 POWER_IN, J9 BYPASS, U10 XL7005A, U11 AP2204K-5.0TRG1, U12 XC6206-1.8NR, U9 XC6206-3.3V

Commit message: Change part number on LCSC for F1/Fuse #172
Parts:
- F1: LCSCStockCode C5183882 -> C2680606
Changed lines of the file:
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@@
       (effects (font (size 1.27 1.27)) hide)
     )
-    (property "LCSCStockCode" "C5183882" (at 48.895 73.025 0)
+    (property "LCSCStockCode" "C2680606" (at 48.895 73.025 0)
       (effects (font (size 1.27 1.27)) hide)
     )
