File: ModuleV490-AllInOne/Module_16S.kicad_sch (KiCad schematic)
At the start: 59 parts, among them J14 BALANCE BOARD, J15 BALANCE BOARD, J6 CELL CONNECTOR PLUG, J7 CELL CONNECTOR, U1 MAX14921ECS+T, U2 MCP1501-40xSN, U3 MCP33151-05-E/MS, U6 MCP1502T-45E/CHY

Commit message: Remove optional footprints
Parts:
- removed JP2: LDO_EN, Jumper:SolderJumper-3_P1.3mm_Bridged12_RoundedPad1.0x1.5mm_NumberLabels, symbol Jumper:SolderJumper_3_Bridged12
- removed U2: MCP1501-40xSN, Package_SO:SOIC-8_3.9x4.9mm_P1.27mm, symbol Reference_Voltage:MCP1501-40xSN
- TP4: value TEST_4096 -> TEST_VREF
- U6: now fitted; now in the parts list
Connections:
- net LDOIN is gone; now on net +5V: U1.13 (LDOIN)
- net VREF4096 renamed VREF

Commit message: Updated part numbers for LCSC 17 pin connector
Parts:
- J6: value CELL CONNECTOR PLUG -> DB2EK-3.81-17P-GN-S; LCSCStockCode C489973 -> C430370; PartNumber WJ15EDGK-3.81-17P -> DB2EK-3.81-17P-GN-S
- J7: LCSCStockCode C489980 -> C430372; PartNumber WJ15EDGRC-3.81-17P -> DB2ERC-3.81-17P-GN
Changed lines of the file:
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@@
       (effects (font (size 1.27 1.27)) hide)
     )
-    (property "PartNumber" "WJ15EDGRC-3.81-17P" (at 168.275 40.64 0)
-      (effects (font (size 1.27 1.27)) hide)
-    )
-    (property "LCSCStockCode" "C489980" (at 168.275 40.64 0)
+    (property "PartNumber" "DB2ERC-3.81-17P-GN" (at 168.275 40.64 0)
+      (effects (font (size 1.27 1.27)) hide)
+    )
+    (property "LCSCStockCode" "C430372" (at 168.275 40.64 0)
       (effects (font (size 1.27 1.27)) hide)
     )
@@
       (effects (font (size 1.27 1.27)) (justify left))
     )
-    (property "Value" "CELL CONNECTOR PLUG" (at 183.515 43.815 90)
+    (property "Value" "DB2EK-3.81-17P-GN-S" (at 183.515 43.815 90)
       (effects (font (size 1.27 1.27)) (justify left))
     )
@@
       (effects (font (size 1.27 1.27)) hide)
     )
-    (property "PartNumber" "WJ15EDGK-3.81-17P" (at 180.975 40.64 0)
+    (property "PartNumber" "DB2EK-3.81-17P-GN-S" (at 180.975 40.64 0)
       (effects (font (size 1.27 1.27)) hide)
     )
@@
       (effects (font (size 1.27 1.27)) hide)
     )
-    (property "LCSCStockCode" "C489973" (at 180.975 40.64 0)
-      (effects (font (size 1.27 1.27)) hide)
-    )
+    (property "LCSCStockCode" "C430370" (at 180.975 40.64 0)
+      (effects (font (size 1.27 1.27)) hide)
+    )
