File: ModuleV490-AllInOne/Module_16S.kicad_sch (KiCad schematic)
At the start: 57 parts, among them J14 BALANCE BOARD, J15 BALANCE BOARD, J6 DB2EK-3.81-17P-GN-S, J7 CELL CONNECTOR, U1 MAX14921ECS+T, U3 MCP33151-05-E/MS, U6 MCP1502T-45E/CHY

Commit message: Add Fiducials
Parts:
- added FID1, FID2, FID3, FID4: Fiducial, Fiducial:Fiducial_1.5mm_Mask3mm, symbol Mechanical:Fiducial
Changed lines of the file:
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@@
+    )
+  )
+  (symbol (lib_id "Mechanical:Fiducial") (at 182.626 135.636 0) (unit 1)
+    (in_bom yes) (on_board yes) (dnp no) (fields_autoplaced)
+    (property "Reference" "FID1" (at 185.42 134.366 0)
+      (effects (font (size 1.27 1.27)) (justify left))
+    )
+    (property "Value" "Fiducial" (at 185.42 136.906 0)
+      (effects (font (size 1.27 1.27)) (justify left))
+    )
+    (property "Footprint" "Fiducial:Fiducial_1.5mm_Mask3mm" (at 182.626 135.636 0)
+      (effects (font (size 1.27 1.27)) hide)
+    )
+    (property "Datasheet" "~" (at 182.626 135.636 0)
+      (effects (font (size 1.27 1.27)) hide)
+    )
+    (instances
+      (project "Module_16S"
+        (path "/e63e39d7-6ac0-4ffd-8aa3-1841a4541b55"
+          (reference "FID1") (unit 1)
+        )
+      )
     )
   )
@@
     )
   )
+  (symbol (lib_id "Mechanical:Fiducial") (at 182.626 139.954 0) (unit 1)
+    (in_bom yes) (on_board yes) (dnp no) (fields_autoplaced)
+    (property "Reference" "FID2" (at 185.42 138.684 0)
+      (effects (font (size 1.27 1.27)) (justify left))
+    )
+    (property "Value" "Fiducial" (at 185.42 141.224 0)
+      (effects (font (size 1.27 1.27)) (justify left))
+    )
+    (property "Footprint" "Fiducial:Fiducial_1.5mm_Mask3mm" (at 182.626 139.954 0)
+      (effects (font (size 1.27 1.27)) hide)
+    )
+    (property "Datasheet" "~" (at 182.626 139.954 0)
+      (effects (font (size 1.27 1.27)) hide)
+    )
+    (instances
+      (project "Module_16S"
+        (path "/e63e39d7-6ac0-4ffd-8aa3-1841a4541b55"
+          (reference "FID2") (unit 1)
+        )
+      )
+    )
+  )
   (symbol (lib_id "Device:R_Small") (at 62.23 49.53 180) (unit 1)
     (in_bom yes) (on_board yes) (dnp no)
@@
         (path "/e63e39d7-6ac0-4ffd-8aa3-1841a4541b55"
           (reference "R5") (unit 1)
+        )
+      )
+    )
+  )
+  (symbol (lib_id "Mechanical:Fiducial") (at 182.626 144.526 0) (unit 1)
+    (in_bom yes) (on_board yes) (dnp no) (fields_autoplaced)
+    (property "Reference" "FID3" (at 185.42 143.256 0)
+      (effects (font (size 1.27 1.27)) (justify left))
+    )
+    (property "Value" "Fiducial" (at 185.42 145.796 0)
+      (effects (font (size 1.27 1.27)) (justify left))
+    )
+    (property "Footprint" "Fiducial:Fiducial_1.5mm_Mask3mm" (at 182.626 144.526 0)
+      (effects (font (size 1.27 1.27)) hide)
+    )
+    (property "Datasheet" "~" (at 182.626 144.526 0)
+      (effects (font (size 1.27 1.27)) hide)
+    )
+    (instances
+      (project "Module_16S"
+        (path "/e63e39d7-6ac0-4ffd-8aa3-1841a4541b55"
+          (reference "FID3") (unit 1)
         )
       )
@@
         )
       )
+    )
+  )
+  (symbol (lib_id "Mechanical:Fiducial") (at 182.626 131.318 0) (unit 1)
+    (in_bom yes) (on_board yes) (dnp no) (fields_autoplaced)
+    (property "Reference" "FID4" (at 185.42 130.048 0)
+      (effects (font (size 1.27 1.27)) (justify left))
+    )
+    (property "Value" "Fiducial" (at 185.42 132.588 0)
+      (effects (font (size 1.27 1.27)) (justify left))
+    )
+    (property "Footprint" "Fiducial:Fiducial_1.5mm_Mask3mm" (at 182.626 131.318 0)
+      (effects (font (size 1.27 1.27)) hide)
+    )
+    (property "Datasheet" "~" (at 182.626 131.318 0)
+      (effects (font (size 1.27 1.27)) hide)
+    )
+    (instances
+      (project "Module_16S"
+        (path "/e63e39d7-6ac0-4ffd-8aa3-1841a4541b55"
+          (reference "FID4") (unit 1)
+        )
+      )

Commit message: Minor part description changes
Parts:
- FID1, FID2, FID3, FID4: now left out of the parts list
- J6: value DB2EK-3.81-17P-GN-S -> MALE PLUG
- U6: LCSCStockCode (none) -> C5236158
Changed lines of the file:
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@@
+      (effects (font (size 1.27 1.27)) hide)
+    )
+    (property "LCSCStockCode" "C5236158" (at 236.855 127 0)
       (effects (font (size 1.27 1.27)) hide)
     )
@@
       (effects (font (size 1.27 1.27)) (justify left))
     )
-    (property "Value" "DB2EK-3.81-17P-GN-S" (at 183.515 43.815 90)
+    (property "Value" "MALE PLUG" (at 183.515 43.815 90)
       (effects (font (size 1.27 1.27)) (justify left))
     )
@@
   )
   (symbol (lib_id "Mechanical:Fiducial") (at 182.626 135.636 0) (unit 1)
-    (in_bom yes) (on_board yes) (dnp no) (fields_autoplaced)
+    (in_bom no) (on_board yes) (dnp no) (fields_autoplaced)
     (property "Reference" "FID1" (at 185.42 134.366 0)
       (effects (font (size 1.27 1.27)) (justify left))
@@
   )
   (symbol (lib_id "Mechanical:Fiducial") (at 182.626 139.954 0) (unit 1)
-    (in_bom yes) (on_board yes) (dnp no) (fields_autoplaced)
+    (in_bom no) (on_board yes) (dnp no) (fields_autoplaced)
     (property "Reference" "FID2" (at 185.42 138.684 0)
       (effects (font (size 1.27 1.27)) (justify left))
@@
   )
   (symbol (lib_id "Mechanical:Fiducial") (at 182.626 144.526 0) (unit 1)
-    (in_bom yes) (on_board yes) (dnp no) (fields_autoplaced)
+    (in_bom no) (on_board yes) (dnp no) (fields_autoplaced)
     (property "Reference" "FID3" (at 185.42 143.256 0)
       (effects (font (size 1.27 1.27)) (justify left))
@@
   )
   (symbol (lib_id "Mechanical:Fiducial") (at 182.626 131.318 0) (unit 1)
-    (in_bom yes) (on_board yes) (dnp no) (fields_autoplaced)
+    (in_bom no) (on_board yes) (dnp no) (fields_autoplaced)
     (property "Reference" "FID4" (at 185.42 130.048 0)
       (effects (font (size 1.27 1.27)) (justify left))

Commit message: Minor tweaks
Parts:
- J6: now left out of the parts list
Changed lines of the file:
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@@
   )
   (symbol (lib_name "Conn_01x17_1") (lib_id "Connector_Generic:Conn_01x17") (at 180.975 40.64 0) (unit 1)
-    (in_bom yes) (on_board no) (dnp no)
+    (in_bom no) (on_board no) (dnp no)
     (property "Reference" "J6" (at 182.88 46.99 0)
       (effects (font (size 1.27 1.27)) (justify left))
