File: ModuleV490-PassiveBal/Module_16S_PassiveBalanceAddOn.kicad_pcb (KiCad board)
At the start: 2 copper layers, 61 x 74 mm, 89 parts, among them J1 FAN_12V, J2 A, J5 B, Q1 AO3400A, Q10 AO3400A, Q11 AO3400A, Q12 AO3400A, Q13 AO3400A, Q14 AO3400A, Q15 AO3400A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

Commit message: Squashed commit of the following:
commit 382df4b7a104fb34cc4a4da3f786b21ade19fcd5
Author: GitHub Action <action@github.com>
Date:   Fri Apr 18 11:47:05 2025 +0000

    CI: pcb-artifacts-ModuleV490-AllInOne

commit b35cb7a0d3894cf57b33edb037eb829bc9ec5ea4
Author: Stuart Pittaway <1201909+stuartpittaway@users.noreply.github.com>
Date:   Fri Apr 18 12:44:57 2025 +0100

    Minor tweaks

commit ea046b7e5d836263693da1b47c6dfb3dc918925c
Author: Stuart Pittaway <1201909+stuartpittaway@users.noreply.github.com>
Date:   Fri Apr 18 12:44:16 2025 +0100

    PCB Panel of Temp sensors

commit ba929f4700586b6858203bc466c6b18e911d661e
Author: GitHub Action <action@github.com>
Date:   Sun Mar 23 15:29:50 2025 +0000

    CI: pcb-artifacts-ModuleV490-AllInOne

commit 1dbbac7378fdc5acb48c43d3f728917ce2318f16
Author: GitHub Action <action@github.com>
Date:   Wed Apr 10 09:57:21 2024 +0000

    CI: pcb-artifacts-ModuleV490-AllInOne

commit 35f617d42fc7a6a7ab395d232005d3307c26595c
Author: Stuart Pittaway <1201909+stuartpittaway@users.noreply.github.com>
Date:   Wed Apr 10 10:55:49 2024 +0100

    Update pcb-artifacts-modulev490-allinone.yaml

commit c8295c0089ea2c5e86742be6a5572142963deb8f
Author: Stuart Pittaway <1201909+stuartpittaway@users.noreply.github.com>
Date:   Wed Apr 10 10:53:50 2024 +0100

    Update pcb-artifacts-modulev490-allinone.yaml

commit d19b2989a6afd4cac4ecf3c8c78554eedba7b99a
Author: Stuart Pittaway <1201909+stuartpittaway@users.noreply.github.com>
Date:   Wed Apr 10 10:50:28 2024 +0100

    Update pcb-artifacts-modulev490-allinone.yaml

commit 8478886fe70d1ee53aca3bbd908099e6f38ff11d
Author: Stuart Pittaway <1201909+stuartpittaway@users.noreply.github.com>
Date:   Wed Apr 10 10:41:28 2024 +0100

    Update pcb-artifacts-modulev490-allinone.yaml

commit afeafa74721a9b51459c6106f0a15ae423229204
Author: Stuart Pittaway <1201909+stuartpittaway@users.noreply.github.com>
Date:   Wed Apr 10 10:39:10 2024 +0100

    Inductor part change - fix workflows

commit 70fd25ba43b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
Parts:
- J1: footprint Connector_JST:JST_PH_B2B-PH-K_1x02_P2.00mm_Vertical -> Connector_JST:JST_PH_B2B-PH-SM4-TB_1x02-1MP_P2.00mm_Vertical
- J2: value A -> 22PIN
- J5: value B -> 22PIN
- moved J1 2.08 mm to (198.9, 78.2), turned to -90 degrees
- moved Q1 0.31 mm to (193.5, 138.0)
- moved Q10 0.31 mm to (193.5, 99.6)
- moved Q11 0.31 mm to (193.5, 95.2)
- moved Q13 0.31 mm to (193.5, 86.8)
- moved Q2 0.31 mm to (193.5, 134.3)
- moved Q3 0.31 mm to (193.5, 130.1)
- moved Q4 0.31 mm to (193.5, 126.0)
- moved Q6 0.31 mm to (193.5, 117.8)
- moved Q7 0.31 mm to (193.5, 113.5)
- moved Q8 0.31 mm to (193.5, 108.6)
- moved Q12 0.30 mm to (193.5, 91.2)
- moved Q5 0.30 mm to (193.5, 121.8)
- moved Q9 0.30 mm to (193.5, 104.5)
- moved R50 0.20 mm to (182.9, 80.3)
Routing:
- net STEP_DOWN_V: track 23.8 -> 28.7 mm
- net Net-(Q16-G): track 27.8 -> 29.4 mm
- net Net-(J1-Pin_2): track 6.33 -> 7.01 mm
- net Net-(Q2-G): track 7.97 -> 8.62 mm
- net GND: vias 87 -> 102
Other:
- board text added: "DIYBMS 8-16S PASSIVE BALANCE BOARD"
- board text removed: "DIYBMS 16S PASSIVE BALANCE BOARD"
