File: ModuleV490-PassiveBal/Module_16S_PassiveBalanceAddOn.kicad_sch (KiCad schematic)
At the start: 9 parts, among them J1 FAN_12V, J2 22PIN, J5 22PIN, Q17 SZNUD3160

Commit message: Squashed commit of the following:
commit 382df4b7a104fb34cc4a4da3f786b21ade19fcd5
Author: GitHub Action <action@github.com>
Date:   Fri Apr 18 11:47:05 2025 +0000

    CI: pcb-artifacts-ModuleV490-AllInOne

commit b35cb7a0d3894cf57b33edb037eb829bc9ec5ea4
Author: Stuart Pittaway <1201909+stuartpittaway@users.noreply.github.com>
Date:   Fri Apr 18 12:44:57 2025 +0100

    Minor tweaks

commit ea046b7e5d836263693da1b47c6dfb3dc918925c
Author: Stuart Pittaway <1201909+stuartpittaway@users.noreply.github.com>
Date:   Fri Apr 18 12:44:16 2025 +0100

    PCB Panel of Temp sensors

commit ba929f4700586b6858203bc466c6b18e911d661e
Author: GitHub Action <action@github.com>
Date:   Sun Mar 23 15:29:50 2025 +0000

    CI: pcb-artifacts-ModuleV490-AllInOne

commit 1dbbac7378fdc5acb48c43d3f728917ce2318f16
Author: GitHub Action <action@github.com>
Date:   Wed Apr 10 09:57:21 2024 +0000

    CI: pcb-artifacts-ModuleV490-AllInOne

commit 35f617d42fc7a6a7ab395d232005d3307c26595c
Author: Stuart Pittaway <1201909+stuartpittaway@users.noreply.github.com>
Date:   Wed Apr 10 10:55:49 2024 +0100

    Update pcb-artifacts-modulev490-allinone.yaml

commit c8295c0089ea2c5e86742be6a5572142963deb8f
Author: Stuart Pittaway <1201909+stuartpittaway@users.noreply.github.com>
Date:   Wed Apr 10 10:53:50 2024 +0100

    Update pcb-artifacts-modulev490-allinone.yaml

commit d19b2989a6afd4cac4ecf3c8c78554eedba7b99a
Author: Stuart Pittaway <1201909+stuartpittaway@users.noreply.github.com>
Date:   Wed Apr 10 10:50:28 2024 +0100

    Update pcb-artifacts-modulev490-allinone.yaml

commit 8478886fe70d1ee53aca3bbd908099e6f38ff11d
Author: Stuart Pittaway <1201909+stuartpittaway@users.noreply.github.com>
Date:   Wed Apr 10 10:41:28 2024 +0100

    Update pcb-artifacts-modulev490-allinone.yaml

commit afeafa74721a9b51459c6106f0a15ae423229204
Author: Stuart Pittaway <1201909+stuartpittaway@users.noreply.github.com>
Date:   Wed Apr 10 10:39:10 2024 +0100

    Inductor part change - fix workflows

commit 70fd25ba43b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
Parts:
- J1: footprint Connector_JST:JST_PH_B2B-PH-K_1x02_P2.00mm_Vertical -> Connector_JST:JST_PH_B2B-PH-SM4-TB_1x02-1MP_P2.00mm_Vertical; LCSCStockCode C265016 -> C2904974; PartNumber S2B-PH-K(LF)(SN) -> B2B-PH-SM4-TB(LF)(SN)
Changed lines of the file:
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@@
       (effects (font (size 1.27 1.27)) (justify left))
     )
-    (property "Footprint" "Connector_JST:JST_PH_B2B-PH-K_1x02_P2.00mm_Vertical" (at 212.725 76.835 0)
+    (property "Footprint" "Connector_JST:JST_PH_B2B-PH-SM4-TB_1x02-1MP_P2.00mm_Vertical" (at 212.725 76.835 0)
       (effects (font (size 1.27 1.27)) hide)
     )
@@
       (effects (font (size 1.27 1.27)) hide)
     )
-    (property "PartNumber" "S2B-PH-K(LF)(SN)" (at 212.725 76.835 0)
+    (property "PartNumber" "B2B-PH-SM4-TB(LF)(SN)" (at 212.725 76.835 0)
       (effects (font (size 1.27 1.27)) hide)
     )
-    (property "LCSCStockCode" "C265016" (at 212.725 76.835 0)
+    (property "LCSCStockCode" "C2904974" (at 212.725 76.835 0)
       (effects (font (size 1.27 1.27)) hide)
     )
