File: TemperaturePCB/TemperaturePCB.kicad_sch (KiCad schematic)
At the start: 3 parts, among them J1 Conn_01x02_Socket

Commit message: Squashed commit of the following:
commit 382df4b7a104fb34cc4a4da3f786b21ade19fcd5
Author: GitHub Action <action@github.com>
Date:   Fri Apr 18 11:47:05 2025 +0000

    CI: pcb-artifacts-ModuleV490-AllInOne

commit b35cb7a0d3894cf57b33edb037eb829bc9ec5ea4
Author: Stuart Pittaway <1201909+stuartpittaway@users.noreply.github.com>
Date:   Fri Apr 18 12:44:57 2025 +0100

    Minor tweaks

commit ea046b7e5d836263693da1b47c6dfb3dc918925c
Author: Stuart Pittaway <1201909+stuartpittaway@users.noreply.github.com>
Date:   Fri Apr 18 12:44:16 2025 +0100

    PCB Panel of Temp sensors

commit ba929f4700586b6858203bc466c6b18e911d661e
Author: GitHub Action <action@github.com>
Date:   Sun Mar 23 15:29:50 2025 +0000

    CI: pcb-artifacts-ModuleV490-AllInOne

commit 1dbbac7378fdc5acb48c43d3f728917ce2318f16
Author: GitHub Action <action@github.com>
Date:   Wed Apr 10 09:57:21 2024 +0000

    CI: pcb-artifacts-ModuleV490-AllInOne

commit 35f617d42fc7a6a7ab395d232005d3307c26595c
Author: Stuart Pittaway <1201909+stuartpittaway@users.noreply.github.com>
Date:   Wed Apr 10 10:55:49 2024 +0100

    Update pcb-artifacts-modulev490-allinone.yaml

commit c8295c0089ea2c5e86742be6a5572142963deb8f
Author: Stuart Pittaway <1201909+stuartpittaway@users.noreply.github.com>
Date:   Wed Apr 10 10:53:50 2024 +0100

    Update pcb-artifacts-modulev490-allinone.yaml

commit d19b2989a6afd4cac4ecf3c8c78554eedba7b99a
Author: Stuart Pittaway <1201909+stuartpittaway@users.noreply.github.com>
Date:   Wed Apr 10 10:50:28 2024 +0100

    Update pcb-artifacts-modulev490-allinone.yaml

commit 8478886fe70d1ee53aca3bbd908099e6f38ff11d
Author: Stuart Pittaway <1201909+stuartpittaway@users.noreply.github.com>
Date:   Wed Apr 10 10:41:28 2024 +0100

    Update pcb-artifacts-modulev490-allinone.yaml

commit afeafa74721a9b51459c6106f0a15ae423229204
Author: Stuart Pittaway <1201909+stuartpittaway@users.noreply.github.com>
Date:   Wed Apr 10 10:39:10 2024 +0100

    Inductor part change - fix workflows

commit 70fd25ba43b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
Parts:
- H1: footprint MountingHole:MountingHole_6.4mm_M6_Pad_Via -> MountingHole:MountingHole_6.5mm_Pad_Via
- J1: value Conn_01x02_Socket -> S2B-PH-SM4-TB(LF)(SN); footprint Connector_PinSocket_2.54mm:PinSocket_1x02_P2.54mm_Vertical -> Connector_JST:JST_PH_S2B-PH-SM4-TB_1x02-1MP_P2.00mm_Horizontal; LCSCStockCode (none) -> C295747
Connections:
- net at J1.1 (Pin_1): now also TH1.2; no longer TH1.1
- net at J1.2 (Pin_2): now also TH1.1; no longer TH1.2
Other:
- moved on the sheet: TH1
Changed lines of the file:
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@@
       (effects (font (size 1.27 1.27)) (justify left))
     )
-    (property "Footprint" "MountingHole:MountingHole_6.4mm_M6_Pad_Via" (at 146.05 96.52 0)
+    (property "Footprint" "MountingHole:MountingHole_6.5mm_Pad_Via" (at 146.05 96.52 0)
       (effects (font (size 1.27 1.27)) hide)
     )
@@
       (effects (font (size 1.27 1.27)) (justify left))
     )
-    (property "Value" "Conn_01x02_Socket" (at 121.92 93.345 90)
+    (property "Value" "S2B-PH-SM4-TB(LF)(SN)" (at 121.92 93.345 90)
       (effects (font (size 1.27 1.27)) (justify left))
     )
-    (property "Footprint" "Connector_PinSocket_2.54mm:PinSocket_1x02_P2.54mm_Vertical" (at 123.19 92.71 0)
+    (property "Footprint" "Connector_JST:JST_PH_S2B-PH-SM4-TB_1x02-1MP_P2.00mm_Horizontal" (at 123.19 92.71 0)
       (effects (font (size 1.27 1.27)) hide)
     )
     (property "Datasheet" "~" (at 123.19 92.71 0)
+      (effects (font (size 1.27 1.27)) hide)
+    )
+    (property "LCSCStockCode" "C295747" (at 123.19 92.71 90)
       (effects (font (size 1.27 1.27)) hide)
     )
@@
     )
   )
-  (symbol (lib_id "Device:Thermistor_NTC") (at 127 74.93 90) (unit 1)
+  (symbol (lib_id "Device:Thermistor_NTC") (at 127 74.93 270) (unit 1)
     (in_bom yes) (on_board yes) (dnp no)
-    (property "Reference" "TH1" (at 127.635 81.28 90)
+    (property "Reference" "TH1" (at 126.365 68.58 90)
       (effects (font (size 1.27 1.27)))
     )
-    (property "Value" "10K NTC" (at 129.54 79.375 90)
+    (property "Value" "10K NTC" (at 124.46 70.485 90)
       (effects (font (size 1.27 1.27)))
     )
-    (property "Footprint" "Resistor_SMD:R_0805_2012Metric" (at 125.73 74.93 0)
+    (property "Footprint" "Resistor_SMD:R_0805_2012Metric" (at 128.27 74.93 0)
       (effects (font (size 1.27 1.27)) hide)
     )
-    (property "Datasheet" "https://datasheet.lcsc.com/szlcsc/Guangdong-Fenghua-Advanced-Tech-CMFB103F3950FANT_C51597.pdf" (at 125.73 74.93 0)
+    (property "Datasheet" "https://datasheet.lcsc.com/szlcsc/Guangdong-Fenghua-Advanced-Tech-CMFB103F3950FANT_C51597.pdf" (at 128.27 74.93 0)
       (effects (font (size 1.27 1.27)) hide)
     )
